File: BuckBoost/alim.kicad_sch (KiCad schematic)
At the start: 23 parts, among them U2 MIC3172YM, U4 MIC3172YM

Commit message: Modifs des conflits
Il y avait des éléments qui avaient les mêmes noms dans le buck et dans le boost du coup ça causait des erreurs
Parts:
- renumbered C1 to C6, C2 to C7, C3 to C8
Changed lines of the file:
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@@
   (symbol (lib_id "Device:C_Small") (at 240.03 86.36 0) (unit 1)
     (in_bom yes) (on_board yes) (dnp no)
-    (property "Reference" "C2" (at 242.57 85.7313 0)
+    (property "Reference" "C7" (at 242.57 85.7313 0)
       (effects (font (size 1.27 1.27)) (justify left))
     )
@@
       (project "alim"
         (path "/9ea535e2-254b-400e-a1b3-21cc38003798"
-          (reference "C2") (unit 1)
+          (reference "C7") (unit 1)
         )
       )
@@
   (symbol (lib_id "Device:C_Small") (at 193.04 88.9 180) (unit 1)
     (in_bom yes) (on_board yes) (dnp no)
-    (property "Reference" "C3" (at 190.5 89.5287 0)
+    (property "Reference" "C8" (at 190.5 89.5287 0)
       (effects (font (size 1.27 1.27)) (justify left))
     )
@@
       (project "alim"
         (path "/9ea535e2-254b-400e-a1b3-21cc38003798"
-          (reference "C3") (unit 1)
+          (reference "C8") (unit 1)
         )
       )
@@
   (symbol (lib_id "Device:C_Small") (at 250.19 60.96 180) (unit 1)
     (in_bom yes) (on_board yes) (dnp no)
-    (property "Reference" "C1" (at 247.65 61.5887 0)
+    (property "Reference" "C6" (at 247.65 61.5887 0)
       (effects (font (size 1.27 1.27)) (justify left))
     )
@@
       (project "alim"
         (path "/9ea535e2-254b-400e-a1b3-21cc38003798"
-          (reference "C1") (unit 1)
-        )
-      )
+          (reference "C6") (unit 1)
+        )
+      )

Commit message: Correction des autres erreurs
Parts:
- renumbered L1 to L2, R3 to R1, R1 to R5, R2 to R6, R3 to R7
Changed lines of the file:
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@@
     (title "alimentation")
   )
+  (junction (at 33.02 38.1) (diameter 0) (color 0 0 0 0)
+  )
   (junction (at 233.68 69.85) (diameter 0) (color 0 0 0 0)
   )
@@
   (junction (at 81.28 96.52) (diameter 0) (color 0 0 0 0)
   )
+  (junction (at 81.28 90.17) (diameter 0) (color 0 0 0 0)
+  )
   (junction (at 54.61 96.52) (diameter 0) (color 0 0 0 0)
   )
@@
   )
   (junction (at 48.26 66.04) (diameter 0) (color 0 0 0 0)
+  )
+  (junction (at 219.71 90.17) (diameter 0) (color 0 0 0 0)
   )
   (junction (at 125.73 107.95) (diameter 0) (color 0 0 0 0)
@@
     (stroke (width 0) (type default))
   )
-  (wire (pts (xy 33.02 44.45) (xy 33.02 36.83))
+  (wire (pts (xy 33.02 44.45) (xy 33.02 38.1))
     (stroke (width 0) (type default))
   )
@@
     (stroke (width 0) (type default))
   )
-  (wire (pts (xy 81.28 86.36) (xy 81.28 96.52))
+  (wire (pts (xy 81.28 86.36) (xy 81.28 90.17))
     (stroke (width 0) (type default))
   )
@@
     (stroke (width 0) (type default))
   )
+  (wire (pts (xy 33.02 38.1) (xy 33.02 36.83))
+    (stroke (width 0) (type default))
+  )
   (wire (pts (xy 233.68 69.85) (xy 234.95 69.85))
     (stroke (width 0) (type default))
@@
   )
   (wire (pts (xy 73.66 86.36) (xy 73.66 96.52))
+    (stroke (width 0) (type default))
+  )
+  (wire (pts (xy 81.28 90.17) (xy 81.28 96.52))
     (stroke (width 0) (type default))
   )
@@
     )
   )
+  (symbol (lib_id "power:PWR_FLAG") (at 33.02 38.1 270) (unit 1)
+    (in_bom yes) (on_board yes) (dnp no) (fields_autoplaced)
+    (property "Reference" "#FLG01" (at 34.925 38.1 0)
+      (effects (font (size 1.27 1.27)) hide)
+    )
+    (property "Value" "PWR_FLAG" (at 36.83 38.735 90)
+      (effects (font (size 1.27 1.27)) (justify left))
+    )
+    (property "Footprint" "" (at 33.02 38.1 0)
+      (effects (font (size 1.27 1.27)) hide)
+    )
+    (property "Datasheet" "~" (at 33.02 38.1 0)
+      (effects (font (size 1.27 1.27)) hide)
+    )
+    (pin "1")
+    (instances
+      (project "alim"
+        (path "/9ea535e2-254b-400e-a1b3-21cc38003798"
+          (reference "#FLG01") (unit 1)
+        )
+      )
+    )
+  )
   (symbol (lib_id "Device:R_Small") (at 193.04 81.28 0) (unit 1)
     (in_bom yes) (on_board yes) (dnp no) (fields_autoplaced)
-    (property "Reference" "R3" (at 195.58 80.645 0)
+    (property "Reference" "R7" (at 195.58 80.645 0)
       (effects (font (size 1.27 1.27)) (justify left))
     )
@@
       (project "alim"
         (path "/9ea535e2-254b-400e-a1b3-21cc38003798"
-          (reference "R3") (unit 1)
+          (reference "R7") (unit 1)
         )
       )
@@
   (symbol (lib_id "Device:R_Small") (at 54.61 82.55 0) (unit 1)
     (in_bom yes) (on_board yes) (dnp no) (fields_autoplaced)
-    (property "Reference" "R3" (at 57.15 81.915 0)
+    (property "Reference" "R1" (at 57.15 81.915 0)
       (effects (font (size 1.27 1.27)) (justify left))
     )
@@
       (project "alim"
         (path "/9ea535e2-254b-400e-a1b3-21cc38003798"
-          (reference "R3") (unit 1)
+          (reference "R1") (unit 1)
         )
       )
@@
   (symbol (lib_id "Device:L_Small") (at 233.68 62.23 0) (unit 1)
     (in_bom yes) (on_board yes) (dnp no)
-    (property "Reference" "L1" (at 231.14 60.96 0)
+    (property "Reference" "L2" (at 231.14 60.96 0)
       (effects (font (size 1.27 1.27)))
     )
@@
       (project "alim"
         (path "/9ea535e2-254b-400e-a1b3-21cc38003798"
-          (reference "L1") (unit 1)
+          (reference "L2") (unit 1)
         )
       )
@@
   (symbol (lib_id "Device:R_Small") (at 250.19 73.66 0) (unit 1)
     (in_bom yes) (on_board yes) (dnp no) (fields_autoplaced)
-    (property "Reference" "R1" (at 252.73 73.025 0)
+    (property "Reference" "R5" (at 252.73 73.025 0)
       (effects (font (size 1.27 1.27)) (justify left))
     )
@@
       (project "alim"
         (path "/9ea535e2-254b-400e-a1b3-21cc38003798"
-          (reference "R1") (unit 1)
+          (reference "R5") (unit 1)
         )
       )
@@
     )
   )
+  (symbol (lib_id "power:PWR_FLAG") (at 219.71 90.17 270) (unit 1)
+    (in_bom yes) (on_board yes) (dnp no) (fields_autoplaced)
+    (property "Reference" "#FLG04" (at 221.615 90.17 0)
+      (effects (font (size 1.27 1.27)) hide)
+    )
+    (property "Value" "PWR_FLAG" (at 223.52 90.805 90)
+      (effects (font (size 1.27 1.27)) (justify left))
+    )
+    (property "Footprint" "" (at 219.71 90.17 0)
+      (effects (font (size 1.27 1.27)) hide)
+    )
+    (property "Datasheet" "~" (at 219.71 90.17 0)
+      (effects (font (size 1.27 1.27)) hide)
+    )
+    (pin "1")
+    (instances
+      (project "alim"
+        (path "/9ea535e2-254b-400e-a1b3-21cc38003798"
+          (reference "#FLG04") (unit 1)
+        )
+      )
+    )
+  )
   (symbol (lib_id "Device:R_Small") (at 125.73 83.82 0) (unit 1)
     (in_bom yes) (on_board yes) (dnp no) (fields_autoplaced)
@@
     )
   )
+  (symbol (lib_id "power:PWR_FLAG") (at 81.28 90.17 270) (unit 1)
+    (in_bom yes) (on_board yes) (dnp no) (fields_autoplaced)
+    (property "Reference" "#FLG02" (at 83.185 90.17 0)
+      (effects (font (size 1.27 1.27)) hide)
+    )
+    (property "Value" "PWR_FLAG" (at 85.09 90.805 90)
+      (effects (font (size 1.27 1.27)) (justify left))
+    )
+    (property "Footprint" "" (at 81.28 90.17 0)
+      (effects (font (size 1.27 1.27)) hide)
+    )
+    (property "Datasheet" "~" (at 81.28 90.17 0)
+      (effects (font (size 1.27 1.27)) hide)
+    )
+    (pin "1")
+    (instances
+      (project "alim"
+        (path "/9ea535e2-254b-400e-a1b3-21cc38003798"
+          (reference "#FLG02") (unit 1)
+        )
+      )
+    )
+  )
   (symbol (lib_id "Device:C_Small") (at 250.19 60.96 180) (unit 1)
     (in_bom yes) (on_board yes) (dnp no)
@@
   (symbol (lib_id "Device:R_Small") (at 250.19 83.82 0) (unit 1)
     (in_bom yes) (on_board yes) (dnp no) (fields_autoplaced)
-    (property "Reference" "R2" (at 252.73 83.185 0)
+    (property "Reference" "R6" (at 252.73 83.185 0)
       (effects (font (size 1.27 1.27)) (justify left))
     )
@@
       (project "alim"
         (path "/9ea535e2-254b-400e-a1b3-21cc38003798"
-          (reference "R2") (unit 1)
-        )
-      )
+          (reference "R6") (unit 1)
+        )
+      )

Commit message: Footprint assignée
Je suis vraiment pas sur pour la diode Shottky
Parts:
- C1, C2, C3, C4, C5, C6, C7, C8: footprint (none) -> Capacitor_SMD:C_0603_1608Metric_Pad1.08x0.95mm_HandSolder
- D1: footprint (none) -> 1N5822:DIOAD2120W130L950D530P
- D2: footprint (none) -> TO-277:TO-277
- D3, D4: footprint (none) -> 1N4148WS-7-F:SOD2513X120N
- L1, L2: footprint (none) -> Inductor_SMD:L_0805_2012Metric_Pad1.05x1.20mm_HandSolder
- R1, R2, R3, R4, R5, R6, R7: footprint (none) -> Resistor_SMD:R_0603_1608Metric_Pad0.98x0.95mm_HandSolder
- U2, U4: footprint SOIC-8_M_MCL -> COHOMA Balise:SOIC127P600X175-8N
Changed lines of the file:
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@@
       (effects (font (size 1.27 1.27)) (justify left))
     )
-    (property "Footprint" "" (at 193.04 81.28 0)
+    (property "Footprint" "Resistor_SMD:R_0603_1608Metric_Pad0.98x0.95mm_HandSolder" (at 193.04 81.28 0)
       (effects (font (size 1.27 1.27)) hide)
     )
@@
       (effects (font (size 1.27 1.27)) (justify left))
     )
-    (property "Footprint" "" (at 114.3 83.82 0)
+    (property "Footprint" "Capacitor_SMD:C_0603_1608Metric_Pad1.08x0.95mm_HandSolder" (at 114.3 83.82 0)
       (effects (font (size 1.27 1.27)) hide)
     )
@@
       (effects (font (size 1.27 1.27)))
     )
-    (property "Footprint" "" (at 119.38 69.85 90)
+    (property "Footprint" "1N4148WS-7-F:SOD2513X120N" (at 119.38 69.85 90)
       (effects (font (size 1.27 1.27)) hide)
     )
@@
       (effects (font (size 1.27 1.27)) (justify left))
     )
-    (property "Footprint" "" (at 54.61 91.44 0)
+    (property "Footprint" "Capacitor_SMD:C_0603_1608Metric_Pad1.08x0.95mm_HandSolder" (at 54.61 91.44 0)
       (effects (font (size 1.27 1.27)) hide)
     )
@@
       (effects (font (size 1.27 1.27)) (justify left))
     )
-    (property "Footprint" "" (at 54.61 82.55 0)
+    (property "Footprint" "Resistor_SMD:R_0603_1608Metric_Pad0.98x0.95mm_HandSolder" (at 54.61 82.55 0)
       (effects (font (size 1.27 1.27)) hide)
     )
@@
       (effects (font (size 1.27 1.27)))
     )
-    (property "Footprint" "" (at 233.68 62.23 0)
+    (property "Footprint" "Inductor_SMD:L_0805_2012Metric_Pad1.05x1.20mm_HandSolder" (at 233.68 62.23 0)
       (effects (font (size 1.27 1.27)) hide)
     )
@@
       (effects (font (size 1.27 1.27)) (justify left))
     )
-    (property "Footprint" "" (at 240.03 86.36 0)
+    (property "Footprint" "Capacitor_SMD:C_0603_1608Metric_Pad1.08x0.95mm_HandSolder" (at 240.03 86.36 0)
       (effects (font (size 1.27 1.27)) hide)
     )
@@
       (effects (font (size 1.27 1.27)) (justify left))
     )
-    (property "Footprint" "" (at 250.19 73.66 0)
+    (property "Footprint" "Resistor_SMD:R_0603_1608Metric_Pad0.98x0.95mm_HandSolder" (at 250.19 73.66 0)
       (effects (font (size 1.27 1.27)) hide)
     )
@@
       (effects (font (size 1.27 1.27)) (justify left))
     )
-    (property "Footprint" "" (at 48.26 72.39 0)
+    (property "Footprint" "Capacitor_SMD:C_0603_1608Metric_Pad1.08x0.95mm_HandSolder" (at 48.26 72.39 0)
       (effects (font (size 1.27 1.27)) hide)
     )
@@
       (effects (font (size 1.27 1.27)) (justify left))
     )
-    (property "Footprint" "" (at 33.02 78.74 0)
+    (property "Footprint" "Capacitor_SMD:C_0603_1608Metric_Pad1.08x0.95mm_HandSolder" (at 33.02 78.74 0)
       (effects (font (size 1.27 1.27)) hide)
     )
@@
       (effects (font (size 1.27 1.27)) (justify left) hide)
     )
-    (property "Footprint" "" (at 114.3 101.6 90)
+    (property "Footprint" "TO-277:TO-277" (at 114.3 101.6 90)
       (effects (font (size 1.27 1.27)) hide)
     )
@@
       (effects (font (size 1.524 1.524)))
     )
-    (property "Footprint" "SOIC-8_M_MCL" (at 236.22 55.88 0)
+    (property "Footprint" "COHOMA Balise:SOIC127P600X175-8N" (at 236.22 55.88 0)
       (effects (font (size 1.524 1.524)) hide)
     )
@@
       (effects (font (size 1.27 1.27)) (justify left))
     )
-    (property "Footprint" "" (at 101.6 83.82 0)
+    (property "Footprint" "Resistor_SMD:R_0603_1608Metric_Pad0.98x0.95mm_HandSolder" (at 101.6 83.82 0)
       (effects (font (size 1.27 1.27)) hide)
     )
@@
       (effects (font (size 1.27 1.27)) (justify left))
     )
-    (property "Footprint" "" (at 193.04 88.9 0)
+    (property "Footprint" "Capacitor_SMD:C_0603_1608Metric_Pad1.08x0.95mm_HandSolder" (at 193.04 88.9 0)
       (effects (font (size 1.27 1.27)) hide)
     )
@@
       (effects (font (size 1.27 1.27)) (justify left))
     )
-    (property "Footprint" "" (at 125.73 101.6 0)
+    (property "Footprint" "Capacitor_SMD:C_0603_1608Metric_Pad1.08x0.95mm_HandSolder" (at 125.73 101.6 0)
       (effects (font (size 1.27 1.27)) hide)
     )
@@
       (effects (font (size 1.27 1.27)) (justify left))
     )
-    (property "Footprint" "" (at 125.73 83.82 0)
+    (property "Footprint" "Resistor_SMD:R_0603_1608Metric_Pad0.98x0.95mm_HandSolder" (at 125.73 83.82 0)
       (effects (font (size 1.27 1.27)) hide)
     )
@@
       (effects (font (size 1.27 1.27)))
     )
-    (property "Footprint" "" (at 119.38 96.52 0)
+    (property "Footprint" "Inductor_SMD:L_0805_2012Metric_Pad1.05x1.20mm_HandSolder" (at 119.38 96.52 0)
       (effects (font (size 1.27 1.27)) hide)
     )
@@
       (effects (font (size 1.27 1.27)))
     )
-    (property "Footprint" "" (at 107.95 69.85 0)
+    (property "Footprint" "Resistor_SMD:R_0603_1608Metric_Pad0.98x0.95mm_HandSolder" (at 107.95 69.85 0)
       (effects (font (size 1.27 1.27)) hide)
     )
@@
       (effects (font (size 1.27 1.27)) (justify left))
     )
-    (property "Footprint" "" (at 250.19 60.96 0)
+    (property "Footprint" "Capacitor_SMD:C_0603_1608Metric_Pad1.08x0.95mm_HandSolder" (at 250.19 60.96 0)
       (effects (font (size 1.27 1.27)) hide)
     )
@@
       (effects (font (size 1.27 1.27)) (justify left))
     )
-    (property "Footprint" "" (at 250.19 83.82 0)
+    (property "Footprint" "Resistor_SMD:R_0603_1608Metric_Pad0.98x0.95mm_HandSolder" (at 250.19 83.82 0)
       (effects (font (size 1.27 1.27)) hide)
     )
@@
       (effects (font (size 1.27 1.27)) (justify right))
     )
-    (property "Footprint" "" (at 76.2 48.26 90)
+    (property "Footprint" "1N4148WS-7-F:SOD2513X120N" (at 76.2 48.26 90)
       (effects (font (size 1.27 1.27)) hide)
     )
@@
       (effects (font (size 1.27 1.27)) (justify left))
     )
-    (property "Footprint" "" (at 237.49 69.85 90)
+    (property "Footprint" "1N5822:DIOAD2120W130L950D530P" (at 237.49 69.85 90)
       (effects (font (size 1.27 1.27)) hide)
     )
@@
       (effects (font (size 1.524 1.524)))
     )
-    (property "Footprint" "SOIC-8_M_MCL" (at 97.79 52.07 0)
+    (property "Footprint" "COHOMA Balise:SOIC127P600X175-8N" (at 97.79 52.07 0)
       (effects (font (size 1.524 1.524)) hide)
     )
