File: BuckBoost/alim-backups/alim-2023-04-16_135933/alim.kicad_pcb (KiCad board)
At the start: 2 copper layers, 35.6 x 33 mm, 24 parts, among them U2 MIC3172YM, U4 MIC3172YM

Commit message: pcb revue
Parts:
- removed D1: 1N5822, Footprints_Balise:DIODE_1N5822-T_DIO
- removed D2: D_Zener_Small, Footprints_Balise:DO-214AD_ONS
- removed D2: D_Zener_Small, TO-277:TO-277
- removed D3, D4: 1N4148, 1N4148WS-7-F:SOD2513X120N
- removed L1: 100 µH, Inductor_SMD:L_0805_2012Metric_Pad1.05x1.20mm_HandSolder
- removed L2: 27 µH, Inductor_SMD:L_0805_2012Metric_Pad1.05x1.20mm_HandSolder
- removed U4: MIC3172YM, COHOMA Balise:SOIC127P600X175-8N
- added C10: 22uF, Capacitor_SMD:CP_Elec_5x5.4, F.Cu at (113.7, 76.0)
- added C9: 470uF, Capacitor_SMD:CP_Elec_10x10.5, F.Cu at (126.0, 47.4)
- added D5: LED, LED_SMD:LED_0603_1608Metric_Pad1.05x0.95mm_HandSolder, F.Cu at (133.9, 54.7)
- added H1: MountingHole_Pad, MountingHole:MountingHole_3.2mm_M3_Pad_Via, F.Cu at (105.2, 45.3)
- added H2: MountingHole_Pad, MountingHole:MountingHole_3.2mm_M3_Pad_Via, F.Cu at (105.2, 53.2)
- added H3: MountingHole_Pad, MountingHole:MountingHole_3.2mm_M3_Pad_Via, F.Cu at (105.2, 61.2)
- added H4: MountingHole_Pad, MountingHole:MountingHole_3.2mm_M3_Pad_Via, F.Cu at (105.2, 69.2)
- added J1: Conn_01x02, Connector_JST:JST_XH_B2B-XH-A_1x02_P2.50mm_Vertical, F.Cu at (112.7, 44.7)
- added J2: Conn_01x02, Connector_JST:JST_XH_B2B-XH-A_1x02_P2.50mm_Vertical, F.Cu at (112.7, 52.5)
- added J3: Conn_01x02, Connector_JST:JST_XH_B2B-XH-A_1x02_P2.50mm_Vertical, F.Cu at (112.7, 60.3)
- added J4: Conn_01x02, Connector_JST:JST_XH_B2B-XH-A_1x02_P2.50mm_Vertical, F.Cu at (112.7, 68.1)
- added R8: 1k, Resistor_SMD:R_0603_1608Metric_Pad0.98x0.95mm_HandSolder, F.Cu at (129.5, 64.7)
- added U1: MIC3172YM, Package_SO:SOIC-8-1EP_3.9x4.9mm_P1.27mm_EP2.29x3mm, F.Cu at (167.5, 56.9)
- C1: value 100 µF -> 0.47u
- C2: value 2.2 µF -> 100uF; footprint Capacitor_SMD:C_0603_1608Metric_Pad1.08x0.95mm_HandSolder -> Capacitor_SMD:CP_Elec_6.3x7.7
- C3: value 1 µF -> 2.2 µF
- C5: value 330 µF -> 0.47u
- C6: value 22 µF -> 1 µF
- C7: value 470 µF -> 330uF
- R5: value 10.7 -> 1k
- R6: value 1.24k -> 10.7
- R7: value 1k -> 1.24k
- U2: footprint COHOMA Balise:SOIC127P600X175-8N -> Package_SO:SOIC-8-1EP_3.9x4.9mm_P1.27mm_EP2.29x3mm
- moved C4 30.5 mm to (120.8, 59.6), turned to 0 degrees
- moved R2 24.7 mm to (125.2, 62.2), turned to 0 degrees
- moved R3 23.7 mm to (125.2, 64.7), turned to 0 degrees
- moved C2 23.0 mm to (132.3, 70.0)
- moved C3 22.2 mm to (120.8, 57.1), turned to 0 degrees
- moved C6 20.0 mm to (120.8, 64.7)
- moved R1 19.0 mm to (125.2, 59.6), turned to 0 degrees
- moved U2 18.2 mm to (122.8, 75.6)
- moved R4 17.2 mm to (129.5, 54.6), turned to 0 degrees
- moved C7 16.2 mm to (125.2, 54.6), turned to 0 degrees
- moved R5 15.1 mm to (129.5, 57.1), turned to 0 degrees
- moved C5 13.0 mm to (120.8, 62.2), turned to 0 degrees
- moved R6 11.1 mm to (129.5, 59.6), turned to 0 degrees
- moved C8 9.58 mm to (125.2, 57.1), turned to 0 degrees
- moved C1 6.65 mm to (120.8, 54.6)
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Connections:
- C1 pad 1: Batteries -> +5V
- C1 pad 2: Earth -> GND
- C2 pad 1: Net-(D4-K) -> +15V
- C2 pad 2: Net-(D2-K) -> Net-(D2-A)
- C3 pad 1: Net-(C3-Pad1) -> Net-(D1-K)
- C3 pad 2: Net-(D2-K) -> GND
- C4 pad 1: Net-(D3-K) -> Net-(C4-Pad1)
- C4 pad 2: Net-(D2-K) -> GND
- C5 pad 1: Camera -> +3.3V
- C5 pad 2: Earth -> GND
- C6 pad 1: Routeur -> Net-(D3-K)
- C6 pad 2: Batteries -> GND
- C7 pad 1: Net-(U2-FB) -> +5V
- C7 pad 2: Earth -> Net-(D2-A)
- C8 pad 1: Earth -> GND
- R1 pad 2: Net-(C3-Pad1) -> Net-(C4-Pad1)
- R2 pad 2: Net-(D2-K) -> GND
- R4 pad 2: Camera -> +5V
- R5 pad 1: Routeur -> Net-(U2-COMP)
- R5 pad 2: Net-(U2-FB) -> Net-(C8-Pad2)
- R6 pad 1: Net-(U2-FB) -> Routeur
- R6 pad 2: Earth -> Net-(U2-FB)
- R7 pad 1: Net-(U2-COMP) -> Net-(U2-FB)
- R7 pad 2: Net-(C8-Pad2) -> GND
- U2 pad 1: Earth -> GND
- U2 pad 5: Batteries -> +15V
- U2 pad 6: Earth -> GND
- U2 pad 8: Earth -> GND
Routing:
- net Batteries: track 50.8 -> 0.00 mm, vias 3 -> 0
- net Earth: track 44.3 -> 0.00 mm, vias 2 -> 0
- net Net-(D2-K): track 42.0 -> 0.00 mm, vias 4 -> 0
- net Net-(D4-A): track 15.8 -> 0.00 mm
- net Net-(U2-FB): track 15.3 -> 0.00 mm
- net Net-(D4-K): track 13.4 -> 0.00 mm
- net Routeur: track 12.9 -> 0.00 mm
- net Camera: track 12.6 -> 0.00 mm
- net Net-(U1-FB): track 10.8 -> 0.00 mm
- net Net-(U2-COMP): track 7.52 -> 0.00 mm
- net Net-(D3-K): track 7.02 -> 0.00 mm
- net Net-(U1-COMP): track 5.41 -> 0.00 mm
- net Net-(D3-A): track 3.55 -> 0.00 mm
- net Net-(C3-Pad1): track 3.07 -> 0.00 mm
- net Net-(C8-Pad2): track 2.49 -> 0.00 mm
- removed copper zone on B.Cu, net (none)
- removed copper zone on F.Cu, net (none)
Other:
- board outline removed
- board text removed: "B"
- board text removed: "BOOST"
- board text removed: "BUCK"
- board text removed: "Balise_Cohoma"
- board text removed: "T"
