File: BuckBoost/alim-backups/alim-2023-04-16_135933/alim.kicad_sch (KiCad schematic)
At the start: 23 parts, among them U2 MIC3172YM, U4 MIC3172YM

Commit message: pcb revue
Parts:
- removed C1: 100 µF, Capacitor_SMD:C_0603_1608Metric_Pad1.08x0.95mm_HandSolder, symbol Device:C_Small
- removed C5: 330 µF, Capacitor_SMD:C_0603_1608Metric_Pad1.08x0.95mm_HandSolder, symbol Device:C_Small
- removed C6: 22 µF, Capacitor_SMD:C_0603_1608Metric_Pad1.08x0.95mm_HandSolder, symbol Device:C_Small
- removed C7: 470 µF, Capacitor_SMD:C_0603_1608Metric_Pad1.08x0.95mm_HandSolder, symbol Device:C_Small
- added C10: 22uF, Capacitor_SMD:CP_Elec_5x5.4, symbol Device:C_Polarized_Small
- added C2: 100uF, Capacitor_SMD:CP_Elec_6.3x7.7, symbol Device:C_Polarized_Small
- added C7: 330uF, Capacitor_SMD:C_0603_1608Metric_Pad1.08x0.95mm_HandSolder, symbol Device:C_Polarized_Small
- added C9: 470uF, Capacitor_SMD:CP_Elec_10x10.5, symbol Device:C_Polarized_Small
- added C? (x2): 0.47u, Capacitor_SMD:C_0603_1608Metric_Pad1.08x0.95mm_HandSolder, symbol Device:C
- added D5: LED, LED_SMD:LED_0603_1608Metric_Pad1.05x0.95mm_HandSolder, symbol Device:LED
- added H1, H2, H3, H4: MountingHole_Pad, MountingHole:MountingHole_3.2mm_M3_Pad_Via, symbol Mechanical:MountingHole_Pad
- added J1, J2, J3, J4: Conn_01x02, Connector_JST:JST_XH_B2B-XH-A_1x02_P2.50mm_Vertical, symbol Connector_Generic:Conn_01x02
- added PS?: BU33SD5WG-TR, Custom:SOT95P280X125-5N, symbol BU33SD5WG-TR:BU33SD5WG-TR
- added R8: 1k, Resistor_SMD:R_0603_1608Metric_Pad0.98x0.95mm_HandSolder, symbol Device:R_Small
- L1, L2: footprint Inductor_SMD:L_0805_2012Metric_Pad1.05x1.20mm_HandSolder -> (none)
- U1: renamed from U4; footprint COHOMA Balise:SOIC127P600X175-8N -> Package_SO:SOIC-8-1EP_3.9x4.9mm_P1.27mm_EP2.29x3mm
- U2: footprint COHOMA Balise:SOIC127P600X175-8N -> Package_SO:SOIC-8-1EP_3.9x4.9mm_P1.27mm_EP2.29x3mm
- renumbered C2 to C3, C3 to C4, C4 to C6, D4 to D1, D1 to D4, R7 to R5, R5 to R6, R6 to R7
Connections:
- net +15V: now also C10.1, C2.1, J4.2 (Pin_2), R8.1
- net Routeur: now also C10.2
- net GND: now reaches C3.2, C4.2, C6.2, D2.1 (K), L1.1, R2.2, U1.1 (SGND), U1.6 (PGND2), U1.8 (PGND1)
- net GND: now also C8.1, R7.2, U2.1 (SGND), U2.6 (PGND2), U2.8 (PGND1), C9.2, C?.2, C?.2, D5.1 (K), H1.1, H2.1, H3.1, H4.1, J1.1 (Pin_1), J2.1 (Pin_1), J3.1 (Pin_1), J4.1 (Pin_1), PS?.2 (GND)
- net at R6.2, R7.1, U2.3 (FB): now also C9.1
- net Camera renamed +5V
- net +5V: now also C7.1, C?.1, J2.2 (Pin_2), J3.2 (Pin_2), PS?.1 (VIN), PS?.3 (STBY)
- removed net Earth: C8.1, D2.2 (A), R7.2, U2.1 (SGND), U2.6 (PGND2), U2.8 (PGND1)
- new net: C2.2, C7.2, D2.2 (A)
- new net: D5.2 (A), R8.2
- new net +3.3V: C?.1, J1.2 (Pin_2), PS?.5 (VOUT)
Other:
- note added: "Input : 12V - 16.8V Output : 5V"

Commit message: ouais
Other:
- note added: "???"
- note added: "LED Test"
- note added: "Mounting Holes"
- moved on the sheet: J1, J2, J3, J4
