File: Hardware/PCB_IR/cohoma.kicad_sch (KiCad schematic)
At the start: 11 parts, among them U1 MCP2120-I/P, U2 TSOP75338WTT, Y1 ABLS-7.3728MHz-20-B-3-H-T

Commit message: PCB IR (le bon)
Parts:
- removed C2: 18 pF, Capacitor_SMD:C_0201_0603Metric_Pad0.64x0.40mm_HandSolder, symbol Device:C
- removed C3: 12 pF, Capacitor_SMD:C_0201_0603Metric_Pad0.64x0.40mm_HandSolder, symbol Device:C
- added C2, C4: 15 pF, Capacitor_SMD:CP_Elec_4x5.7, symbol Device:C_Polarized_Small
- added H4: Mounting Hole 4, MountingHole:MountingHole_3.2mm_M3_DIN965_Pad, symbol Mechanical:MountingHole_Pad
- C1: value 7 pF -> 4.7 pF; footprint Capacitor_SMD:C_0603_1608Metric_Pad1.08x0.95mm_HandSolder -> Capacitor_SMD:CP_Elec_4x5.4
- H1: value Alimentation -> Mounting Hole 1; footprint MountingHole:MountingHole_4.3mm_M4_ISO14580_Pad_TopOnly -> MountingHole:MountingHole_3.2mm_M3_DIN965_Pad
- H2: renamed from H3; value UART_RX -> Mounting Hole 2; footprint MountingHole:MountingHole_2.2mm_M2_DIN965_Pad -> MountingHole:MountingHole_3.2mm_M3_DIN965_Pad
- H3: renamed from H4; value UART_TX -> Mounting Hole 3; footprint MountingHole:MountingHole_2.2mm_M2_DIN965_Pad -> MountingHole:MountingHole_3.2mm_M3_DIN965_Pad
- U1: footprint TerminalBlock_4Ucon:TerminalBlock_4Ucon_1x14_P3.50mm_Horizontal -> Package_SO:SOIC-8-N7_3.9x4.9mm_P1.27mm
- U2: footprint (none) -> Capacitor_SMD:CP_Elec_4x5.4
- Y1: footprint Resistor_SMD:R_0201_0603Metric_Pad0.64x0.40mm_HandSolder -> Crystal:Crystal_SMD_EuroQuartz_MQ-4Pin_7.0x5.0mm
Connections:
- net +3.3V: no longer C1.2, H1.1, H2.1, H3.1, U1.11 (RX), U1.12 (TX), U1.14 (VSS), U2.1 (GND), U2.4 (GND)
- net at R1.1, Y1.2: now also C4.1
- net at R2.1, U2.2 (VS): now also C2.1
- new net GND: C1.2, C2.2, C4.2, H1.1, H2.1, H3.1, H4.1, U1.14 (VSS), U2.1 (GND), U2.4 (GND)
- new net UART_RX: U1.11 (RX)
- new net UART_TX: U1.12 (TX)

Commit message: IR
Parts:
- removed C2: 15 pF, Capacitor_SMD:CP_Elec_4x5.7, symbol Device:C_Polarized_Small
- added C2: 0,1 pF, symbol Device:C
- added J1: Conn_01x02, symbol Connector_Generic:Conn_01x02
Connections:
- net GND: now also C2.2
- net UART_RX: now also J1.2 (Pin_2)
- net UART_TX: now also J1.1 (Pin_1)
- net at R2.1, U2.2 (VS): now also C2.1
Other:
- note added: "Mounting holes"
- note removed: "Mounting hole"
- title: Cohoma -> Cohoma IR
- moved on the sheet: H2, H3
Changed lines of the file:
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@@
   (paper "A4")
   (title_block
-    (title "Cohoma")
+    (title "Cohoma IR")
   )
   (junction (at 148.59 95.25) (diameter 0) (color 0 0 0 0)
   )
+  (junction (at 148.59 76.2) (diameter 0) (color 0 0 0 0)
+  )
+  (junction (at 160.02 153.67) (diameter 0) (color 0 0 0 0)
+  )
   (junction (at 209.55 128.27) (diameter 0) (color 0 0 0 0)
   )
-  (junction (at 148.59 87.63) (diameter 0) (color 0 0 0 0)
+  (junction (at 148.59 85.09) (diameter 0) (color 0 0 0 0)
   )
   (junction (at 245.11 66.04) (diameter 0) (color 0 0 0 0)
@@
   )
   (junction (at 195.58 140.97) (diameter 0) (color 0 0 0 0)
-  )
-  (junction (at 148.59 77.47) (diameter 0) (color 0 0 0 0)
   )
   (junction (at 34.29 85.09) (diameter 0) (color 0 0 0 0)
@@
     (stroke (width 0) (type default))
   )
-  (wire (pts (xy 148.59 64.77) (xy 148.59 77.47))
+  (wire (pts (xy 148.59 64.77) (xy 148.59 76.2))
     (stroke (width 0) (type default))
   )
@@
     (stroke (width 0) (type default))
   )
-  (wire (pts (xy 209.55 139.7) (xy 209.55 143.51))
+  (wire (pts (xy 160.02 153.67) (xy 173.99 153.67))
     (stroke (width 0) (type default))
   )
@@
     (stroke (width 0) (type default))
   )
-  (wire (pts (xy 154.94 153.67) (xy 173.99 153.67))
+  (wire (pts (xy 154.94 153.67) (xy 160.02 153.67))
     (stroke (width 0) (type default))
   )
@@
     (stroke (width 0) (type default))
   )
-  (wire (pts (xy 148.59 77.47) (xy 148.59 87.63))
-    (stroke (width 0) (type default))
-  )
   (wire (pts (xy 245.11 66.04) (xy 257.81 66.04))
     (stroke (width 0) (type default))
@@
     (stroke (width 0) (type default))
   )
+  (wire (pts (xy 148.59 85.09) (xy 148.59 95.25))
+    (stroke (width 0) (type default))
+  )
   (wire (pts (xy 257.81 58.42) (xy 257.81 66.04))
     (stroke (width 0) (type default))
@@
     (stroke (width 0) (type default))
   )
-  (wire (pts (xy 148.59 87.63) (xy 149.86 87.63))
+  (wire (pts (xy 148.59 85.09) (xy 149.86 85.09))
     (stroke (width 0) (type default))
   )
@@
     (stroke (width 0) (type default))
   )
-  (polyline (pts (xy 246.38 120.65) (xy 246.38 158.75))
+  (wire (pts (xy 209.55 142.24) (xy 209.55 143.51))
+    (stroke (width 0) (type default))
+  )
+  (polyline (pts (xy 246.38 116.84) (xy 246.38 160.02))
     (stroke (width 0) (type default))
   )
@@
     (stroke (width 0) (type default))
   )
-  (wire (pts (xy 148.59 87.63) (xy 148.59 95.25))
-    (stroke (width 0) (type default))
-  )
   (wire (pts (xy 196.85 128.27) (xy 209.55 128.27))
+    (stroke (width 0) (type default))
+  )
+  (wire (pts (xy 148.59 76.2) (xy 148.59 85.09))
     (stroke (width 0) (type default))
   )
@@
     (effects (font (size 1.27 1.27)) (justify left bottom))
   )
-  (text "Mounting hole" (at 123.19 50.8 0)
+  (text "Mounting holes" (at 123.19 50.8 0)
     (effects (font (size 1.27 1.27)) (justify left bottom))
   )
@@
     )
   )
+  (global_label "UART_RX" (shape input) (at 67.31 158.75 0) (fields_autoplaced)
+    (effects (font (size 1.27 1.27)) (justify left))
+    (property "Intersheetrefs" "${INTERSHEET_REFS}" (at 78.3196 158.75 0)
+      (effects (font (size 1.27 1.27)) (justify left) hide)
+    )
+  )
   (global_label "UART_RX" (shape input) (at 82.55 92.71 0) (fields_autoplaced)
     (effects (font (size 1.27 1.27)) (justify left))
@@
     )
   )
+  (global_label "UART_TX" (shape input) (at 67.31 161.29 0) (fields_autoplaced)
+    (effects (font (size 1.27 1.27)) (justify left))
+    (property "Intersheetrefs" "${INTERSHEET_REFS}" (at 78.0172 161.29 0)
+      (effects (font (size 1.27 1.27)) (justify left) hide)
+    )
+  )
   (symbol (lib_id "power:PWR_FLAG") (at 34.29 85.09 0) (unit 1)
     (in_bom yes) (on_board yes) (dnp no) (fields_autoplaced)
@@
     )
   )
-  (symbol (lib_id "Device:C_Polarized_Small") (at 209.55 137.16 0) (unit 1)
-    (in_bom yes) (on_board yes) (dnp no) (fields_autoplaced)
-    (property "Reference" "C2" (at 212.09 135.9789 0)
-      (effects (font (size 1.27 1.27)) (justify left))
-    )
-    (property "Value" "15 pF" (at 212.09 138.5189 0)
-      (effects (font (size 1.27 1.27)) (justify left))
-    )
-    (property "Footprint" "Capacitor_SMD:CP_Elec_4x5.7" (at 209.55 137.16 0)
-      (effects (font (size 1.27 1.27)) hide)
-    )
-    (property "Datasheet" "~" (at 209.55 137.16 0)
+  (symbol (lib_id "Device:C") (at 209.55 138.43 0) (unit 1)
+    (in_bom yes) (on_board yes) (dnp no) (fields_autoplaced)
+    (property "Reference" "C2" (at 213.36 137.795 0)
+      (effects (font (size 1.27 1.27)) (justify left))
+    )
+    (property "Value" "0,1 pF" (at 213.36 140.335 0)
+      (effects (font (size 1.27 1.27)) (justify left))
+    )
+    (property "Footprint" "" (at 210.5152 142.24 0)
+      (effects (font (size 1.27 1.27)) hide)
+    )
+    (property "Datasheet" "~" (at 209.55 138.43 0)
       (effects (font (size 1.27 1.27)) hide)
     )
@@
     )
   )
-  (symbol (lib_id "Mechanical:MountingHole_Pad") (at 151.13 77.47 270) (unit 1)
-    (in_bom yes) (on_board yes) (dnp no) (fields_autoplaced)
-    (property "Reference" "H2" (at 154.94 76.835 90)
-      (effects (font (size 1.27 1.27)) (justify left))
-    )
-    (property "Value" "Mounting Hole 2" (at 154.94 79.375 90)
-      (effects (font (size 1.27 1.27)) (justify left))
-    )
-    (property "Footprint" "MountingHole:MountingHole_3.2mm_M3_DIN965_Pad" (at 151.13 77.47 0)
-      (effects (font (size 1.27 1.27)) hide)
-    )
-    (property "Datasheet" "~" (at 151.13 77.47 0)
+  (symbol (lib_id "Mechanical:MountingHole_Pad") (at 151.13 76.2 270) (unit 1)
+    (in_bom yes) (on_board yes) (dnp no) (fields_autoplaced)
+    (property "Reference" "H2" (at 154.94 75.565 90)
+      (effects (font (size 1.27 1.27)) (justify left))
+    )
+    (property "Value" "Mounting Hole 2" (at 154.94 78.105 90)
+      (effects (font (size 1.27 1.27)) (justify left))
+    )
+    (property "Footprint" "MountingHole:MountingHole_3.2mm_M3_DIN965_Pad" (at 151.13 76.2 0)
+      (effects (font (size 1.27 1.27)) hide)
+    )
+    (property "Datasheet" "~" (at 151.13 76.2 0)
       (effects (font (size 1.27 1.27)) hide)
     )
@@
     )
   )
-  (symbol (lib_id "Mechanical:MountingHole_Pad") (at 152.4 87.63 270) (unit 1)
-    (in_bom yes) (on_board yes) (dnp no) (fields_autoplaced)
-    (property "Reference" "H3" (at 156.21 86.995 90)
-      (effects (font (size 1.27 1.27)) (justify left))
-    )
-    (property "Value" "Mounting Hole 3" (at 156.21 89.535 90)
-      (effects (font (size 1.27 1.27)) (justify left))
-    )
-    (property "Footprint" "MountingHole:MountingHole_3.2mm_M3_DIN965_Pad" (at 152.4 87.63 0)
-      (effects (font (size 1.27 1.27)) hide)
-    )
-    (property "Datasheet" "~" (at 152.4 87.63 0)
+  (symbol (lib_id "Mechanical:MountingHole_Pad") (at 152.4 85.09 270) (unit 1)
+    (in_bom yes) (on_board yes) (dnp no) (fields_autoplaced)
+    (property "Reference" "H3" (at 156.21 84.455 90)
+      (effects (font (size 1.27 1.27)) (justify left))
+    )
+    (property "Value" "Mounting Hole 3" (at 156.21 86.995 90)
+      (effects (font (size 1.27 1.27)) (justify left))
+    )
+    (property "Footprint" "MountingHole:MountingHole_3.2mm_M3_DIN965_Pad" (at 152.4 85.09 0)
+      (effects (font (size 1.27 1.27)) hide)
+    )
+    (property "Datasheet" "~" (at 152.4 85.09 0)
       (effects (font (size 1.27 1.27)) hide)
     )
@@
         )
       )
+    )
+  )
+  (symbol (lib_id "power:PWR_FLAG") (at 160.02 153.67 0) (unit 1)
+    (in_bom yes) (on_board yes) (dnp no) (fields_autoplaced)
+    (property "Reference" "#FLG03" (at 160.02 151.765 0)
+      (effects (font (size 1.27 1.27)) hide)
+    )
+    (property "Value" "PWR_FLAG" (at 160.02 149.86 0)
+      (effects (font (size 1.27 1.27)))
+    )
+    (property "Footprint" "" (at 160.02 153.67 0)
+      (effects (font (size 1.27 1.27)) hide)
+    )
+    (property "Datasheet" "~" (at 160.02 153.67 0)
+      (effects (font (size 1.27 1.27)) hide)
+    )
+    (pin "1")
+    (instances
+      (project "cohoma"
+        (path "/b67a6078-ca99-4579-a5b2-eb9bf477316b"
+          (reference "#FLG03") (unit 1)
+        )
+      )
+    )
+  )
+  (symbol (lib_id "Connector_Generic:Conn_01x02") (at 62.23 161.29 180) (unit 1)
+    (in_bom yes) (on_board yes) (dnp no) (fields_autoplaced)
+    (property "Reference" "J1" (at 62.23 153.67 0)
+      (effects (font (size 1.27 1.27)))
+    )
+    (property "Value" "Conn_01x02" (at 62.23 156.21 0)
+      (effects (font (size 1.27 1.27)))
+    )
+    (property "Footprint" "" (at 62.23 161.29 0)
+      (effects (font (size 1.27 1.27)) hide)
+    )
+    (property "Datasheet" "~" (at 62.23 161.29 0)
+      (effects (font (size 1.27 1.27)) hide)
+    )
+    (pin "1")
+    (pin "2")
+    (instances
+      (project "cohoma"
+        (path "/b67a6078-ca99-4579-a5b2-eb9bf477316b"
+          (reference "J1") (unit 1)
+        )
+      )

Commit message: PCB IR
Parts:
- removed C4: 15 pF, Capacitor_SMD:CP_Elec_4x5.7, symbol Device:C_Polarized_Small
- removed J1: Conn_01x02, symbol Connector_Generic:Conn_01x02
- removed R1: 500 M, Resistor_SMD:R_0201_0603Metric_Pad0.64x0.40mm_HandSolder, symbol Device:R
- removed R2: 30k, Resistor_SMD:R_0201_0603Metric_Pad0.64x0.40mm_HandSolder, symbol Device:R
- added C3: 20 pF, Capacitor_SMD:CP_Elec_4x5.4, symbol Device:C
- added J2: Conn_01x03, symbol Connector_Generic:Conn_01x03
- C1: value 4.7 pF -> 20 pF
- C2: value 0,1 pF -> 100 nF
Connections:
- net +3.3V: now also C2.1, U1.13 (EN), U1.4 (*RESET), U2.2 (VS), J2.3 (Pin_3)
- net GND: now also U1.10 (BAUD0), U1.8 (BAUD2), U1.9 (BAUD1), C3.2, J2.1 (Pin_1)
- net Q_OUT: now also Y1.2, C3.1
- net UART_RX: now also J2.2 (Pin_2)
- net UART_TX: no longer names the net of U1.12 (TX)
- no-connect marks 7 -> 3
Other:
- moved on the sheet: H1, H2, H3, H4, U1
