File: Hardware/BuckBoost/alim-backups/alim-2023-04-16_135933/alim.kicad_sch (KiCad schematic)
At the start: 36 parts, among them J1 Conn_01x02, J2 Conn_01x02, J3 Conn_01x02, J4 Conn_01x02, U1 MIC3172YM, U2 MIC3172YM

Commit message: PPZ m'as aidé
Parts:
- PS?: footprint Custom:SOT95P280X125-5N -> footprints:SSOP5_ROM
Changed lines of the file:
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@@
       (effects (font (size 1.27 1.27)))
     )
-    (property "Footprint" "Custom:SOT95P280X125-5N" (at 34.29 161.29 0)
+    (property "Footprint" "footprints:SSOP5_ROM" (at 34.29 161.29 0)
       (effects (font (size 1.27 1.27)) (justify left bottom) hide)
     )

Commit message: renommage des datasheets et assignation d'empreintes du Buck/Boost
Parts:
- D1: footprint Footprints_Balise:SOD2513X120N -> Diode_SMD:D_SOD-123F
- D2: value D_Zener_Small -> FSV330AF
- D3: footprint Footprints_Balise:SOD2513X120N -> Diode_SMD:D_SOD-323F
- D4: value 1N5822 -> FSV330AF
- L1: footprint (none) -> Inductor_SMD_Wurth:L_Wurth_WE-LQSH-2512
- L2: value 27 µH -> 120 µH; footprint (none) -> Inductor_SMD_Wurth:L_Wurth_WE-LQSH-2512
Changed lines of the file:
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@@
       (effects (font (size 1.27 1.27)))
     )
-    (property "Footprint" "Footprints_Balise:SOD2513X120N" (at 119.38 69.85 90)
+    (property "Footprint" "Diode_SMD:D_SOD-323F" (at 119.38 69.85 90)
       (effects (font (size 1.27 1.27)) hide)
     )
@@
       (effects (font (size 1.27 1.27)))
     )
-    (property "Value" "27 µH" (at 229.87 63.5 0)
-      (effects (font (size 1.27 1.27)))
-    )
-    (property "Footprint" "" (at 233.68 62.23 0)
+    (property "Value" "120 µH" (at 229.87 63.5 0)
+      (effects (font (size 1.27 1.27)))
+    )
+    (property "Footprint" "Inductor_SMD_Wurth:L_Wurth_WE-LQSH-2512" (at 233.68 62.23 0)
       (effects (font (size 1.27 1.27)) hide)
     )
@@
       (effects (font (size 1.27 1.27)) (justify left))
     )
-    (property "Value" "D_Zener_Small" (at 116.84 103.505 90)
-      (effects (font (size 1.27 1.27)) (justify left) hide)
+    (property "Value" "FSV330AF" (at 102.87 104.14 90)
+      (effects (font (size 1.27 1.27)) (justify left))
     )
     (property "Footprint" "Footprints_Balise:DO-214AD_ONS" (at 114.3 101.6 90)
@@
       (effects (font (size 1.27 1.27)))
     )
-    (property "Footprint" "" (at 119.38 96.52 0)
+    (property "Footprint" "Inductor_SMD_Wurth:L_Wurth_WE-LQSH-2512" (at 119.38 96.52 0)
       (effects (font (size 1.27 1.27)) hide)
     )
@@
       (effects (font (size 1.27 1.27)) (justify right))
     )
-    (property "Footprint" "Footprints_Balise:SOD2513X120N" (at 76.2 48.26 90)
+    (property "Footprint" "Diode_SMD:D_SOD-123F" (at 76.2 48.26 90)
       (effects (font (size 1.27 1.27)) hide)
     )
@@
       (effects (font (size 1.27 1.27)) (justify left))
     )
-    (property "Value" "1N5822" (at 241.3 72.39 0)
-      (effects (font (size 1.27 1.27)) (justify left))
-    )
+    (property "Value" "FSV330AF" (at 241.3 72.39 0)
+      (effects (font (size 1.27 1.27)) (justify left))
+    )

Commit message: composants ps1 associé
Parts:
- PS?: footprint footprints:SSOP5_ROM -> Footprints_Balise:SSOP5_ROM
Changed lines of the file:
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@@
       (effects (font (size 1.27 1.27)))
     )
-    (property "Footprint" "footprints:SSOP5_ROM" (at 34.29 161.29 0)
+    (property "Footprint" "Footprints_Balise:SSOP5_ROM" (at 34.29 161.29 0)
       (effects (font (size 1.27 1.27)) (justify left bottom) hide)
     )
