File: Hardware/PCB_BuckBoost/kicad_alim/alim.kicad_sch (KiCad schematic)
At the start: 36 parts, among them J1 Conn_01x02, J2 Conn_01x02, J3 Conn_01x02, J4 Conn_01x02, U1 MIC3172YM, U2 MIC3172YM

Commit message: assignation d'empreintes
Parts:
- C?: footprint diode:SSOP5_ROM -> Capacitor_SMD:C_0603_1608Metric
- PS?: footprint diode:SSOP5_ROM -> custom:ssop5
Changed lines of the file:
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@@
       (effects (font (size 1.27 1.27)))
     )
-    (property "Footprint" "diode:SSOP5_ROM" (at 34.29 161.29 0)
+    (property "Footprint" "custom:ssop5" (at 34.29 161.29 0)
       (effects (font (size 1.27 1.27)) (justify left bottom) hide)
     )
@@
       (effects (font (size 1.27 1.27)) (justify left))
     )
-    (property "Footprint" "diode:SSOP5_ROM" (at 20.0152 156.21 0)
+    (property "Footprint" "Capacitor_SMD:C_0603_1608Metric" (at 20.0152 156.21 0)
       (effects (font (size 1.27 1.27)) hide)
     )
