File: Hardware/PCB_BuckBoost/kicad_alim/alim.kicad_sch (KiCad schematic)
At the start: 36 parts, among them J1 Conn_01x02, J2 Conn_01x02, J3 Conn_01x02, J4 Conn_01x02, U1 MIC3172YM, U2 MIC3172YM

Commit message: Réparé ?
Parts:
- D2, D4: footprint custom:Diode_Shottky -> Custom_BUCKBOOST:Diode_Shottky
- PS?: footprint custom:ssop5 -> Custom_BUCKBOOST:ssop5
Changed lines of the file:
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@@
       (effects (font (size 1.27 1.27)))
     )
-    (property "Footprint" "custom:ssop5" (at 34.29 161.29 0)
+    (property "Footprint" "Custom_BUCKBOOST:ssop5" (at 34.29 161.29 0)
       (effects (font (size 1.27 1.27)) (justify left bottom) hide)
     )
@@
       (effects (font (size 1.27 1.27)) (justify left))
     )
-    (property "Footprint" "custom:Diode_Shottky" (at 114.3 101.6 90)
+    (property "Footprint" "Custom_BUCKBOOST:Diode_Shottky" (at 114.3 101.6 90)
       (effects (font (size 1.27 1.27)) hide)
     )
@@
       (effects (font (size 1.27 1.27)) (justify left))
     )
-    (property "Footprint" "custom:Diode_Shottky" (at 237.49 69.85 90)
-      (effects (font (size 1.27 1.27)) hide)
-    )
+    (property "Footprint" "Custom_BUCKBOOST:Diode_Shottky" (at 237.49 69.85 90)
+      (effects (font (size 1.27 1.27)) hide)
+    )

Commit message: a
Parts:
- D2, D4: footprint Custom_BUCKBOOST:Diode_Shottky -> Custom_BUCKBOOST:Diode_Shottky (copy)
- PS?: footprint Custom_BUCKBOOST:ssop5 -> Custom_BUCKBOOST:ssop5 (copy)
Changed lines of the file:
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@@
       (effects (font (size 1.27 1.27)))
     )
-    (property "Footprint" "Custom_BUCKBOOST:ssop5" (at 34.29 161.29 0)
+    (property "Footprint" "Custom_BUCKBOOST:ssop5 (copy)" (at 34.29 161.29 0)
       (effects (font (size 1.27 1.27)) (justify left bottom) hide)
     )
@@
       (effects (font (size 1.27 1.27)) (justify left))
     )
-    (property "Footprint" "Custom_BUCKBOOST:Diode_Shottky" (at 114.3 101.6 90)
+    (property "Footprint" "Custom_BUCKBOOST:Diode_Shottky (copy)" (at 114.3 101.6 90)
       (effects (font (size 1.27 1.27)) hide)
     )
@@
       (effects (font (size 1.27 1.27)) (justify left))
     )
-    (property "Footprint" "Custom_BUCKBOOST:Diode_Shottky" (at 237.49 69.85 90)
-      (effects (font (size 1.27 1.27)) hide)
-    )
+    (property "Footprint" "Custom_BUCKBOOST:Diode_Shottky (copy)" (at 237.49 69.85 90)
+      (effects (font (size 1.27 1.27)) hide)
+    )

Commit message: routage pcb
Parts:
- C7: footprint Capacitor_SMD:C_0603_1608Metric_Pad1.08x0.95mm_HandSolder -> Capacitor_SMD:CP_Elec_10x10.5
Changed lines of the file:
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@@
       (effects (font (size 1.27 1.27)) (justify left))
     )
-    (property "Footprint" "Capacitor_SMD:C_0603_1608Metric_Pad1.08x0.95mm_HandSolder" (at 125.73 101.6 0)
+    (property "Footprint" "Capacitor_SMD:CP_Elec_10x10.5" (at 125.73 101.6 0)
       (effects (font (size 1.27 1.27)) hide)
     )

Commit message: PCB Final en avancement
Parts:
- PS?: footprint Custom_BUCKBOOST:ssop5 (copy) -> Package_TO_SOT_SMD:TSOT-23-5_HandSoldering
Changed lines of the file:
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@@
       (effects (font (size 1.27 1.27)))
     )
-    (property "Footprint" "Custom_BUCKBOOST:ssop5 (copy)" (at 34.29 161.29 0)
+    (property "Footprint" "Package_TO_SOT_SMD:TSOT-23-5_HandSoldering" (at 34.29 161.29 0)
       (effects (font (size 1.27 1.27)) (justify left bottom) hide)
     )
