File: Hardware/PCB_BuckBoost/kicad_alim/alim.kicad_pcb (KiCad board)
At the start: 2 copper layers, 58.4 x 58.4 mm, 36 parts, among them J1 Conn_01x02, J2 Conn_01x02, J3 Conn_01x02, J4 Conn_01x02, U1 MIC3172YM, U2 MIC3172YM

Commit message: routage pcb
Parts:
- C7: footprint Capacitor_SMD:C_0603_1608Metric_Pad1.08x0.95mm_HandSolder -> Capacitor_SMD:CP_Elec_10x10.5
- moved C2 117.3 mm to (181.6, 75.9), turned to 180 degrees
- moved C3 115.4 mm to (183.0, 92.6), turned to 180 degrees
- moved C4 115.2 mm to (183.0, 94.1)
- moved D3 113.4 mm to (175.4, 88.6)
- moved R2 110.7 mm to (183.0, 95.6)
- moved C6 110.5 mm to (179.6, 92.6)
- moved R1 107.7 mm to (179.7, 94.1)
- moved D2 107.4 mm to (180.1, 75.5)
- moved R3 103.3 mm to (176.3, 94.1), turned to 180 degrees
- moved R4 102.5 mm to (176.3, 92.6), turned to 180 degrees
- moved C7 100.4 mm to (171.1, 82.2)
- moved U1 90.3 mm to (181.9, 84.1)
