File: Hardware/PCB_BuckBoost/kicad_alim/alim.kicad_pcb (KiCad board)
At the start: 2 copper layers, 36 parts, among them J1 Conn_01x02, J2 Conn_01x02, J3 Conn_01x02, J4 Conn_01x02, U1 MIC3172YM, U2 MIC3172YM

Commit message: pcb presque terminé (3 erreurs)
Parts:
- moved PS1 84.4 mm to (77.8, 87.6), turned to 180 degrees
- moved D3 66.8 mm to (88.9, 83.8), turned to 90 degrees
- moved U1 61.2 mm to (114.9, 88.2)
- moved D4 57.9 mm to (96.5, 53.3), turned to -90 degrees
- moved R7 56.0 mm to (73.7, 58.4), turned to -90 degrees
- moved C1 54.2 mm to (86.4, 96.5)
- moved H2 53.0 mm to (127.0, 101.6)
- moved C9 48.8 mm to (81.3, 66.9), turned to -90 degrees
- moved J1 48.2 mm to (76.2, 76.2), turned to -90 degrees
- moved R6 45.8 mm to (83.8, 55.9), turned to -90 degrees
- moved H4 43.4 mm to (76.2, 101.5)
- moved R3 43.0 mm to (91.4, 91.4), turned to 180 degrees
- moved D2 41.9 mm to (119.4, 104.1), turned to 180 degrees
- moved J3 41.8 mm to (106.7, 101.6), turned to 180 degrees
- moved L1 40.6 mm to (113.4, 101.6)
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Routing:
- net GND: track 0.00 -> 158.3 mm, vias 0 -> 6
- net +5V: track 0.00 -> 112.1 mm, vias 0 -> 2
- net +15V: track 0.00 -> 75.7 mm
- net Routeur: track 0.00 -> 39.0 mm
- net Net-(U2-FB): track 0.00 -> 27.4 mm
- net Net-(D2-A): track 0.00 -> 25.8 mm, vias 0 -> 2
- net Net-(D4-A): track 0.00 -> 25.1 mm
- net Net-(U1-FB): track 0.00 -> 22.4 mm
- net +3.3V: track 0.00 -> 20.0 mm
- net Net-(D3-K): track 0.00 -> 19.3 mm
- net Net-(D1-K): track 0.00 -> 17.6 mm
- net Net-(D3-A): track 0.00 -> 15.8 mm
- net Net-(D5-A): track 0.00 -> 6.71 mm
- net Net-(C4-Pad1): track 0.00 -> 6.64 mm
- net Net-(C8-Pad2): track 0.00 -> 6.49 mm
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- added copper zone on F.Cu, net GND
Other:
- board outline added: 61 x 61 mm

Commit message: j'ai corrigé les erreurs dans le pcb
Routing:
- net +15V: track 75.7 -> 86.9 mm
- net +5V: track 112.1 -> 120.5 mm
- net GND: track 158.3 -> 155.8 mm
Changed lines of the file:
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@@
   (segment (start 89.615 63.5) (end 88.235 64.88) (width 0.25) (layer "F.Cu") (net 6))
   (segment (start 101.6 75.41) (end 101.6 73.66) (width 0.25) (layer "F.Cu") (net 8))
+  (segment (start 106.68 101.64) (end 106.72 101.6) (width 0.25) (layer "F.Cu") (net 8))
   (segment (start 96.405 68.465) (end 96.52 68.58) (width 0.25) (layer "F.Cu") (net 8))
-  (segment (start 115.7204 105.5604) (end 112.55 102.39) (width 0.25) (layer "F.Cu") (net 8))
   (segment (start 93.98 62.6375) (end 89.7625 58.42) (width 0.25) (layer "F.Cu") (net 8))
   (segment (start 103.5483 50.2083) (end 76.7917 50.2083) (width 0.25) (layer "F.Cu") (net 8))
   (segment (start 106.68 91.44) (end 104.14 93.98) (width 0.25) (layer "F.Cu") (net 8))
   (segment (start 104.14 50.8) (end 103.5483 50.2083) (width 0.25) (layer "F.Cu") (net 8))
-  (segment (start 127 101.6) (end 123.0396 105.5604) (width 0.25) (layer "F.Cu") (net 8))
+  (segment (start 106.72 101.6) (end 112.55 101.6) (width 0.25) (layer "F.Cu") (net 8))
+  (segment (start 83.82 73.66) (end 81.28 71.12) (width 0.25) (layer "F.Cu") (net 8))
   (segment (start 102.39 76.2) (end 100.7375 77.8525) (width 0.25) (layer "F.Cu") (net 8))
   (segment (start 127 76.2) (end 130.2 73) (width 0.25) (layer "F.Cu") (net 8))
+  (segment (start 83.82 77.8775) (end 83.82 73.66) (width 0.25) (layer "F.Cu") (net 8))
   (segment (start 100.7375 77.8525) (end 100.7375 80.4175) (width 0.25) (layer "F.Cu") (net 8))
   (segment (start 93.98 65.42) (end 94.485 65.925) (width 0.25) (layer "F.Cu") (net 8))
   (segment (start 93.98 63.5) (end 93.98 65.42) (width 0.25) (layer "F.Cu") (net 8))
   (segment (start 117.345 88.785) (end 119.265 88.785) (width 0.25) (layer "F.Cu") (net 8))
+  (segment (start 122.06 104.14) (end 124.6 101.6) (width 0.25) (layer "F.Cu") (net 8))
   (segment (start 112.55 102.39) (end 112.55 101.6) (width 0.25) (layer "F.Cu") (net 8))
   (segment (start 94.485 68.465) (end 96.405 68.465) (width 0.25) (layer "F.Cu") (net 8))
@@
   (segment (start 116.84 83.82) (end 114.82 83.82) (width 0.25) (layer "F.Cu") (net 8))
   (segment (start 114.82 83.82) (end 112.395 86.245) (width 0.25) (layer "F.Cu") (net 8))
-  (segment (start 124.46 104.14) (end 121.6152 104.14) (width 0.25) (layer "F.Cu") (net 8))
   (segment (start 130.2 54) (end 127 50.8) (width 0.25) (layer "F.Cu") (net 8))
   (segment (start 127 101.6) (end 124.46 104.14) (width 0.25) (layer "F.Cu") (net 8))
-  (segment (start 123.0396 105.5604) (end 115.7204 105.5604) (width 0.25) (layer "F.Cu") (net 8))
   (segment (start 106.68 91.44) (end 106.78 91.44) (width 0.25) (layer "F.Cu") (net 8))
   (segment (start 130.2 73) (end 130.2 54) (width 0.25) (layer "F.Cu") (net 8))
   (segment (start 112.395 86.245) (end 117.345 86.245) (width 0.25) (layer "F.Cu") (net 8))
   (segment (start 102.39 76.2) (end 101.6 75.41) (width 0.25) (layer "F.Cu") (net 8))
+  (segment (start 121.6152 104.14) (end 122.06 104.14) (width 0.25) (layer "F.Cu") (net 8))
   (segment (start 94.485 65.925) (end 89.535 65.925) (width 0.25) (layer "F.Cu") (net 8))
   (segment (start 93.98 63.5) (end 93.98 62.6375) (width 0.25) (layer "F.Cu") (net 8))
@@
   (segment (start 96.52 66.04) (end 93.98 63.5) (width 0.25) (layer "B.Cu") (net 8))
   (segment (start 96.52 68.58) (end 96.52 66.04) (width 0.25) (layer "B.Cu") (net 8))
-  (segment (start 117.1448 104.14) (end 117.1448 102.9375) (width 0.25) (layer "F.Cu") (net 9))
+  (segment (start 117.1448 104.14) (end 117.1448 102.6293) (width 0.25) (layer "F.Cu") (net 9))
   (segment (start 124.46 93.98) (end 127 91.44) (width 0.25) (layer "F.Cu") (net 9))
   (segment (start 127 91.44) (end 127 89.06) (width 0.25) (layer "F.Cu") (net 9))
@@
   (segment (start 116.84 102.3245) (end 116.84 101.6) (width 0.25) (layer "B.Cu") (net 9))
   (segment (start 78.7123 88.5444) (end 78.3134 88.1455) (width 0.25) (layer "F.Cu") (net 10))
+  (segment (start 104.18 101.64) (end 99.06 96.52) (width 0.25) (layer "F.Cu") (net 10))
+  (segment (start 121.92 101.6) (end 129.54 93.98) (width 0.25) (layer "F.Cu") (net 10))
   (segment (start 85.0646 95.5802) (end 85.0646 94.5134) (width 0.25) (layer "F.Cu") (net 10))
-  (segment (start 129.54 93.98) (end 121.92 101.6) (width 0.25) (layer "F.Cu") (net 10))
+  (segment (start 114.3 101.075) (end 114.3 101.6) (width 0.25) (layer "F.Cu") (net 10))
+  (segment (start 99.06 96.52) (end 86.36 96.52) (width 0.25) (layer "F.Cu") (net 10))
   (segment (start 78.3134 87.2057) (end 78.8543 86.6648) (width 0.25) (layer "F.Cu") (net 10))
-  (segment (start 84.7598 95.5802) (end 85.0646 95.5802) (width 0.25) (layer "F.Cu") (net 10))
-  (segment (start 83.82 96.52) (end 84.7598 95.5802) (width 0.25) (layer "F.Cu") (net 10))
   (segment (start 92.1004 73.66) (end 79.0956 86.6648) (width 0.25) (layer "F.Cu") (net 10))
-  (segment (start 104.18 101.64) (end 87.9217 101.64) (width 0.25) (layer "F.Cu") (net 10))
-  (segment (start 87.9217 101.64) (end 83.82 97.5383) (width 0.25) (layer "F.Cu") (net 10))
-  (segment (start 121.92 101.6) (end 114.3 101.6) (width 0.25) (layer "F.Cu") (net 10))
+  (segment (start 114.3 101.6) (end 121.92 101.6) (width 0.25) (layer "F.Cu") (net 10))
+  (segment (start 86.36 96.52) (end 85.4202 95.5802) (width 0.25) (layer "F.Cu") (net 10))
   (segment (start 99.06 71.12) (end 99.06 72.7475) (width 0.25) (layer "F.Cu") (net 10))
   (segment (start 78.3134 88.1455) (end 78.3134 87.2057) (width 0.25) (layer "F.Cu") (net 10))
+  (segment (start 104.18 101.64) (end 105.545 100.275) (width 0.25) (layer "F.Cu") (net 10))
+  (segment (start 113.5 100.275) (end 114.3 101.075) (width 0.25) (layer "F.Cu") (net 10))
   (segment (start 79.0956 88.5444) (end 78.7123 88.5444) (width 0.25) (layer "F.Cu") (net 10))
+  (segment (start 105.545 100.275) (end 113.5 100.275) (width 0.25) (layer "F.Cu") (net 10))
   (segment (start 78.8543 86.6648) (end 79.0956 86.6648) (width 0.25) (layer "F.Cu") (net 10))
-  (segment (start 83.82 97.5383) (end 83.82 96.52) (width 0.25) (layer "F.Cu") (net 10))
   (segment (start 106.64 50.8) (end 109.22 50.8) (width 0.25) (layer "F.Cu") (net 10))
   (segment (start 98.1475 73.66) (end 92.1004 73.66) (width 0.25) (layer "F.Cu") (net 10))
@@
   (segment (start 99.06 72.7475) (end 98.1475 73.66) (width 0.25) (layer "F.Cu") (net 10))
   (segment (start 85.0646 94.5134) (end 79.0956 88.5444) (width 0.25) (layer "F.Cu") (net 10))
+  (segment (start 85.4202 95.5802) (end 85.0646 95.5802) (width 0.25) (layer "F.Cu") (net 10))
   (via (at 111.76 53.34) (size 0.8) (drill 0.4) (layers "F.Cu" "B.Cu") (net 10))
   (via (at 99.06 71.12) (size 0.8) (drill 0.4) (layers "F.Cu" "B.Cu") (net 10))
@@
   (segment (start 116.84 72.0325) (end 116.84 66.04) (width 0.25) (layer "F.Cu") (net 11))
   (segment (start 107.205 69.455) (end 110.62 66.04) (width 0.25) (layer "F.Cu") (net 11))
+  (segment (start 125.539897 75.160103) (end 125.539897 82.199897) (width 0.25) (layer "F.Cu") (net 11))
   (segment (start 110.62 66.04) (end 116.84 66.04) (width 0.25) (layer "F.Cu") (net 11))
   (segment (start 124.5 73.7) (end 116.84 66.04) (width 0.25) (layer "F.Cu") (net 11))
@@
   (segment (start 94.765 69.455) (end 94.485 69.735) (width 0.25) (layer "F.Cu") (net 11))
   (segment (start 127 73.7) (end 124.5 73.7) (width 0.25) (layer "F.Cu") (net 11))
+  (segment (start 125.539897 82.199897) (end 127 83.66) (width 0.25) (layer "F.Cu") (net 11))
   (segment (start 117.345 87.515) (end 117.36 87.5) (width 0.25) (layer "F.Cu") (net 11))
   (segment (start 123.16 87.5) (end 127 83.66) (width 0.25) (layer "F.Cu") (net 11))
+  (segment (start 127 73.7) (end 125.539897 75.160103) (width 0.25) (layer "F.Cu") (net 11))
   (segment (start 121.92 87.5) (end 123.16 87.5) (width 0.25) (layer "F.Cu") (net 11))
   (segment (start 117.36 87.5) (end 121.92 87.5) (width 0.25) (layer "F.Cu") (net 11))
@@
   (segment (start 102.415 83.82) (end 106.68 83.82) (width 0.25) (layer "F.Cu") (net 13))
   (segment (start 76.2 81.28) (end 73.66 83.82) (width 0.25) (layer "F.Cu") (net 14))
+  (segment (start 76.2 78.74) (end 82.9575 78.74) (width 0.25) (layer "F.Cu") (net 14))
   (segment (start 73.66 83.82) (end 73.66 85.7123) (width 0.25) (layer "F.Cu") (net 14))
-  (segment (start 82.9575 78.74) (end 76.2 78.74) (width 0.25) (layer "F.Cu") (net 14))
-  (segment (start 83.82 79.6025) (end 82.9575 78.74) (width 0.25) (layer "F.Cu") (net 14))
+  (segment (start 82.9575 78.74) (end 83.82 79.6025) (width 0.25) (layer "F.Cu") (net 14))
   (segment (start 73.66 85.7123) (end 76.5048 88.5571) (width 0.25) (layer "F.Cu") (net 14))
   (segment (start 76.2 78.74) (end 76.2 81.28) (width 0.25) (layer "F.Cu") (net 14))

Commit message: a
Parts:
- C1: footprint diode:SSOP5_ROM -> Capacitor_SMD:C_0603_1608Metric
- D2, D4: footprint Footprints_Balise:DO-214AD_ONS -> Custom_BUCKBOOST:Diode_Shottky (copy)
- L2: value 120 µH -> 27 µH
- PS1: footprint diode:SSOP5_ROM -> Custom_BUCKBOOST:ssop5 (copy)
- moved R7 96.1 mm to (168.2, 75.6), turned to 0 degrees
- moved R6 86.1 mm to (168.2, 73.1), turned to 0 degrees
- moved D4 82.7 mm to (167.9, 95.0), turned to 0 degrees
- moved R5 78.0 mm to (168.2, 70.6)
- moved C9 78.0 mm to (156.3, 88.2), turned to 0 degrees
- moved C8 75.9 mm to (163.8, 70.6), turned to 0 degrees
- moved C5 75.7 mm to (159.5, 75.6), turned to 0 degrees
- moved C1 75.3 mm to (161.3, 103.4)
- moved R3 73.6 mm to (163.8, 78.1), turned to 0 degrees
- moved J1 66.8 mm to (142.9, 72.7), turned to 0 degrees
- moved R2 65.7 mm to (163.8, 75.6), turned to 0 degrees
- moved D3 65.3 mm to (151.0, 103.9), turned to 0 degrees
- moved R4 65.1 mm to (163.8, 80.6), turned to 0 degrees
- moved H1 63.4 mm to (135.4, 73.3)
- moved U2 62.1 mm to (153.1, 79.0)
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Connections:
- C2 pad 2: Net-(D2-A) -> GND
- C3 pad 2: GND -> Net-(D2-K)
- C4 pad 2: GND -> Net-(D2-K)
- C6 pad 2: GND -> Net-(D2-K)
- C7 pad 2: Net-(D2-A) -> GND
- C9 pad 1: Net-(U2-FB) -> Routeur
- D2 pad 1: GND -> Net-(D2-K)
- D2 pad 2: Net-(D2-A) -> GND
- L1 pad 1: GND -> Net-(D2-K)
- R2 pad 2: GND -> Net-(D2-K)
- U1 pad 1: GND -> Net-(D2-K)
- U1 pad 6: GND -> Net-(D2-K)
- U1 pad 8: GND -> Net-(D2-K)
Routing:
- net GND: track 155.8 -> 0.00 mm, vias 6 -> 0
- net +5V: track 120.5 -> 0.00 mm, vias 2 -> 0
- net +15V: track 86.9 -> 0.00 mm
- net Routeur: track 39.0 -> 0.00 mm
- net Net-(U2-FB): track 27.4 -> 0.00 mm
- net Net-(D2-A): track 26.1 -> 0.00 mm, vias 2 -> 0
- net Net-(D4-A): track 25.1 -> 0.00 mm
- net Net-(U1-FB): track 22.4 -> 0.00 mm
- net +3.3V: track 20.0 -> 0.00 mm
- net Net-(D3-K): track 19.3 -> 0.00 mm
- net Net-(D1-K): track 17.6 -> 0.00 mm
- net Net-(D3-A): track 15.8 -> 0.00 mm
- net Net-(D5-A): track 6.71 -> 0.00 mm
- net Net-(C4-Pad1): track 6.64 -> 0.00 mm
- net Net-(C8-Pad2): track 6.49 -> 0.00 mm
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- removed copper zone on F.Cu, net GND
Other:
- board size 61 x 61 mm -> 3 x 3 mm

Commit message: b
Parts:
- moved U1 31.8 mm to (180.1, 89.3)
Changed lines of the file:
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@@
   )
   (footprint "Package_SO:SOIC-8-1EP_3.9x4.9mm_P1.27mm_EP2.29x3mm" (layer "F.Cu")
-    (at 153.076 72.54)
+    (at 180.148 89.269)
     (descr "SOIC, 8 Pin (https://www.analog.com/media/en/technical-documentation/data-sheets/ada4898-1_4898-2.pdf#page=29), generated with kicad-footprint-generator ipc_gullwing_generator.py")
     (tags "SOIC SO")

Commit message: OUi
Parts:
- moved U2 53.3 mm to (206.3, 82.0)
Changed lines of the file:
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@@
   )
   (footprint "Package_SO:SOIC-8-1EP_3.9x4.9mm_P1.27mm_EP2.29x3mm" (layer "F.Cu")
-    (at 153.076 78.99)
+    (at 206.31 82.03)
     (descr "SOIC, 8 Pin (https://www.analog.com/media/en/technical-documentation/data-sheets/ada4898-1_4898-2.pdf#page=29), generated with kicad-footprint-generator ipc_gullwing_generator.py")
     (tags "SOIC SO")

Commit message: début du routage pcb
Parts:
- moved U2 114.0 mm to (92.7, 72.7)
- moved C1 88.7 mm to (72.7, 98.0)
- moved C10 88.7 mm to (55.3, 98.5)
- moved J1 88.7 mm to (54.3, 67.3)
- moved J2 88.7 mm to (54.3, 75.1)
- moved J3 88.7 mm to (54.3, 82.9)
- moved J4 88.7 mm to (54.3, 90.7)
- moved L1 88.7 mm to (77.0, 78.6)
- moved L2 88.7 mm to (77.0, 82.2)
- moved C2 88.7 mm to (65.5, 92.9)
- moved C3 88.7 mm to (70.9, 65.1)
- moved C4 88.7 mm to (70.9, 67.6)
- moved C5 88.7 mm to (70.9, 70.2)
- moved C6 88.7 mm to (70.9, 72.7)
- moved C7 88.7 mm to (70.9, 75.2)
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Routing:
- added copper zone on B.Cu, net GND
- added copper zone on F.Cu, net GND
Other:
- board size 3 x 3 mm -> 58.4 x 58.4 mm

Commit message: ok
Parts:
- moved C9 106.9 mm to (171.8, 107.1), turned to 90 degrees
- moved C10 102.1 mm to (157.4, 98.2)
- moved L2 89.5 mm to (161.8, 110.7), turned to 90 degrees
- moved R5 87.8 mm to (156.3, 107.8)
- moved R7 87.8 mm to (156.3, 112.8)
- moved R6 87.8 mm to (156.3, 110.3)
- moved C8 87.8 mm to (152.0, 107.8)
- moved D4 87.8 mm to (167.0, 94.6)
- moved U2 76.6 mm to (162.5, 104.3)
- moved R8 20.7 mm to (79.9, 93.3)
Changed lines of the file:
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@@
   (net 19 "unconnected-(U2-SYNC{slash}EN-Pad4)")
   (footprint "Resistor_SMD:R_0603_1608Metric_Pad0.98x0.95mm_HandSolder" (layer "F.Cu")
-    (at 79.615 65.134)
+    (at 156.3351 107.8114)
     (descr "Resistor SMD 0603 (1608 Metric), square (rectangular) end terminal, IPC_7351 nominal with elongated pad for handsoldering. (Body size source: IPC-SM-782 page 72, https://www.pcb-3d.com/wordpress/wp-content/uploads/ipc-sm-782a_amendment_1_and_2.pdf), generated with kicad-footprint-generator")
     (tags "resistor handsolder")
@@
   )
   (footprint "Capacitor_SMD:CP_Elec_10x10.5" (layer "F.Cu")
-    (at 67.7 82.804)
+    (at 171.7802 107.0954 90)
     (descr "SMD capacitor, aluminum electrolytic, Vishay 1010, 10.0x10.5mm, http://www.vishay.com/docs/28395/150crz.pdf")
     (tags "capacitor electrolytic")
@@
     (property "ki_keywords" "cap capacitor")
     (attr smd)
-    (fp_text reference "C9" (at 0 -6.3) (layer "F.SilkS")
-        (effects (font (size 1 1) (thickness 0.15)))
-    )
-    (fp_text value "470uF" (at 0 6.3) (layer "F.Fab")
-        (effects (font (size 1 1) (thickness 0.15)))
-    )
-    (fp_text user "${REFERENCE}" (at 0 0) (layer "F.Fab")
+    (fp_text reference "C9" (at 0 -6.3 90) (layer "F.SilkS")
+        (effects (font (size 1 1) (thickness 0.15)))
+    )
+    (fp_text value "470uF" (at 0 6.3 90) (layer "F.Fab")
+        (effects (font (size 1 1) (thickness 0.15)))
+    )
+    (fp_text user "${REFERENCE}" (at 0 0 90) (layer "F.Fab")
         (effects (font (size 1 1) (thickness 0.15)))
     )
@@
     (fp_circle (center 0 0) (end 5 0)
       (stroke (width 0.1) (type solid)) (fill none) (layer "F.Fab"))
-    (pad "1" smd roundrect (at -4.2 0) (size 4.4 2.5) (layers "F.Cu" "F.Paste" "F.Mask") (roundrect_rratio 0.1)
+    (pad "1" smd roundrect (at -4.2 0 90) (size 4.4 2.5) (layers "F.Cu" "F.Paste" "F.Mask") (roundrect_rratio 0.1)
       (net 10 "Routeur") (pintype "passive"))
-    (pad "2" smd roundrect (at 4.2 0) (size 4.4 2.5) (layers "F.Cu" "F.Paste" "F.Mask") (roundrect_rratio 0.1)
+    (pad "2" smd roundrect (at 4.2 0 90) (size 4.4 2.5) (layers "F.Cu" "F.Paste" "F.Mask") (roundrect_rratio 0.1)
       (net 2 "GND") (pintype "passive"))
     (model "${KICAD6_3DMODEL_DIR}/Capacitor_SMD.3dshapes/CP_Elec_10x10.5.wrl"
@@
   )
   (footprint "Capacitor_SMD:CP_Elec_5x5.4" (layer "F.Cu")
-    (at 55.315 98.504)
+    (at 157.423 98.233)
     (descr "SMD capacitor, aluminum electrolytic, Nichicon, 5.0x5.4mm")
     (tags "capacitor electrolytic")
@@
   )
   (footprint "Resistor_SMD:R_0603_1608Metric_Pad0.98x0.95mm_HandSolder" (layer "F.Cu")
-    (at 79.615 70.154)
+    (at 156.3351 112.8314)
     (descr "Resistor SMD 0603 (1608 Metric), square (rectangular) end terminal, IPC_7351 nominal with elongated pad for handsoldering. (Body size source: IPC-SM-782 page 72, https://www.pcb-3d.com/wordpress/wp-content/uploads/ipc-sm-782a_amendment_1_and_2.pdf), generated with kicad-footprint-generator")
     (tags "resistor handsolder")
@@
   )
   (footprint "Package_SO:SOIC-8-1EP_3.9x4.9mm_P1.27mm_EP2.29x3mm" (layer "F.Cu")
-    (at 92.73 72.669)
+    (at 162.495 104.2924)
     (descr "SOIC, 8 Pin (https://www.analog.com/media/en/technical-documentation/data-sheets/ada4898-1_4898-2.pdf#page=29), generated with kicad-footprint-generator ipc_gullwing_generator.py")
     (tags "SOIC SO")
@@
         (effects (font (size 1 1) (thickness 0.15)))
     )
-    (fp_text value "MIC3172YM" (at 0 3.4) (layer "F.Fab")
+    (fp_text value "MIC3172YM" (at -8.3932 -5.3086 90) (layer "F.Fab")
         (effects (font (size 1 1) (thickness 0.15)))
     )
@@
   )
   (footprint "Custom_BUCKBOOST:Diode_Shottky (copy)" (layer "F.Cu")
-    (at 79.365 89.579)
+    (at 166.9984 94.5728)
     (property "Sheetfile" "alim.kicad_sch")
     (property "Sheetname" "")
@@
   )
   (footprint "Capacitor_SMD:C_0603_1608Metric_Pad1.08x0.95mm_HandSolder" (layer "F.Cu")
-    (at 75.265 65.134)
+    (at 151.9851 107.8114)
     (descr "Capacitor SMD 0603 (1608 Metric), square (rectangular) end terminal, IPC_7351 nominal with elongated pad for handsoldering. (Body size source: IPC-SM-782 page 76, https://www.pcb-3d.com/wordpress/wp-content/uploads/ipc-sm-782a_amendment_1_and_2.pdf), generated with kicad-footprint-generator")
     (tags "capacitor handsolder")
@@
   )
   (footprint "Resistor_SMD:R_0603_1608Metric_Pad0.98x0.95mm_HandSolder" (layer "F.Cu")
-    (at 79.615 72.664)
+    (at 79.8849 93.345)
     (descr "Resistor SMD 0603 (1608 Metric), square (rectangular) end terminal, IPC_7351 nominal with elongated pad for handsoldering. (Body size source: IPC-SM-782 page 72, https://www.pcb-3d.com/wordpress/wp-content/uploads/ipc-sm-782a_amendment_1_and_2.pdf), generated with kicad-footprint-generator")
     (tags "resistor handsolder")
@@
   )
   (footprint "Inductor_SMD_Wurth:L_Wurth_WE-LQSH-2512" (layer "F.Cu")
-    (at 76.995 82.239)
+    (at 161.798 110.7072 90)
     (descr "Semi-Shielded High Saturation Power Inductor, body 2.5x2mm, https://www.we-online.com/catalog/en/WE-LQSH#/articles/WE-LQSH-2512")
     (tags "SMT")
@@
     (property "ki_keywords" "inductor choke coil reactor magnetic")
     (attr smd)
-    (fp_text reference "L2" (at 0 -2 unlocked) (layer "F.SilkS")
-        (effects (font (size 1 1) (thickness 0.15)))
-    )
-    (fp_text value "27 µH" (at 0 2.1 unlocked) (layer "F.Fab")
-        (effects (font (size 1 1) (thickness 0.15)))
-    )
-    (fp_text user "${REFERENCE}" (at 0 0 unlocked) (layer "F.Fab")
+    (fp_text reference "L2" (at 0 -2 90 unlocked) (layer "F.SilkS")
+        (effects (font (size 1 1) (thickness 0.15)))
+    )
+    (fp_text value "27 µH" (at 0 2.1 90 unlocked) (layer "F.Fab")
+        (effects (font (size 1 1) (thickness 0.15)))
+    )
+    (fp_text user "${REFERENCE}" (at 0 0 90 unlocked) (layer "F.Fab")
         (effects (font (size 0.5 0.5) (thickness 0.075)))
     )
@@
     (fp_line (start 1.25 -1) (end 1.25 1)
       (stroke (width 0.1) (type solid)) (layer "F.Fab"))
-    (pad "1" smd rect (at -0.875 0) (size 0.95 2) (layers "F.Cu" "F.Paste" "F.Mask")
+    (pad "1" smd rect (at -0.875 0 90) (size 0.95 2) (layers "F.Cu" "F.Paste" "F.Mask")
       (net 3 "+15V") (pintype "passive"))
-    (pad "2" smd rect (at 0.875 0) (size 0.95 2) (layers "F.Cu" "F.Paste" "F.Mask")
+    (pad "2" smd rect (at 0.875 0 90) (size 0.95 2) (layers "F.Cu" "F.Paste" "F.Mask")
       (net 12 "Net-(D4-A)") (pintype "passive"))
     (model "${KICAD6_3DMODEL_DIR}/Inductor_SMD_Wurth.3dshapes/L_Wurth_WE-LQSH-2512.wrl"
@@
   )
   (footprint "Resistor_SMD:R_0603_1608Metric_Pad0.98x0.95mm_HandSolder" (layer "F.Cu")
-    (at 79.615 67.644)
+    (at 156.3351 110.3214)
     (descr "Resistor SMD 0603 (1608 Metric), square (rectangular) end terminal, IPC_7351 nominal with elongated pad for handsoldering. (Body size source: IPC-SM-782 page 72, https://www.pcb-3d.com/wordpress/wp-content/uploads/ipc-sm-782a_amendment_1_and_2.pdf), generated with kicad-footprint-generator")
     (tags "resistor handsolder")
@@
     (connect_pads (clearance 0.5))
     (min_thickness 0.25) (filled_areas_thickness no)
-    (fill (thermal_gap 0.5) (thermal_bridge_width 0.5))
+    (fill yes (thermal_gap 0.5) (thermal_bridge_width 0.5))
     (polygon
       (pts
