File: Hardware/PCB_IR/cohoma-backups/cohoma-2023-05-03_234336/cohoma.kicad_pcb (KiCad board)
At the start: 2 copper layers, 32.9 x 32.6 mm, 11 parts, among them J2 Conn_01x03, U1 MCP2120-I/P, U2 TSOP75338WTT, Y1 ABLS-7.3728MHz-20-B-3-H-T

Commit message: essai
Parts:
- moved J2 0.67 mm to (122.0, 79.3)
Routing:
- net +3.3V: track 113.3 -> 104.1 mm, vias 3 -> 2
- net Q_OUT: track 20.1 -> 21.6 mm
Other:
- board text removed: "B"
- board text removed: "Maëna CHARBONNIER"
- board text removed: "T"
Changed lines of the file:
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@@
     (property "ki_keywords" "cap capacitor")
     (attr smd)
-    (fp_text reference "C3" (at 1 1.36) (layer "F.SilkS")
+    (fp_text reference "C3" (at 0 -3.2) (layer "F.SilkS")
         (effects (font (size 1 1) (thickness 0.15)))
     )
@@
         (effects (font (size 1 1) (thickness 0.15)))
     )
-    (fp_text value "ABLS-7.3728MHz-20-B-3-H-T" (at -21.21 1.51) (layer "F.Fab")
+    (fp_text value "ABLS-7.3728MHz-20-B-3-H-T" (at -18.52 3.7) (layer "F.Fab")
         (effects (font (size 1 1) (thickness 0.15)))
     )
@@
     (property "ki_keywords" "cap capacitor")
     (attr smd)
-    (fp_text reference "C1" (at 0.33 1.28) (layer "F.SilkS")
+    (fp_text reference "C1" (at 0 -3.2) (layer "F.SilkS")
         (effects (font (size 1 1) (thickness 0.15)))
     )
@@
     (property "ki_keywords" "cap capacitor")
     (attr smd)
-    (fp_text reference "C2" (at 0.32 -3.07) (layer "F.SilkS")
+    (fp_text reference "C2" (at -1.195563 -2.26) (layer "F.SilkS")
         (effects (font (size 1 1) (thickness 0.15)))
     )
@@
   )
   (footprint "Connector_PinHeader_1.27mm:PinHeader_1x03_P1.27mm_Horizontal" (layer "F.Cu")
-    (at 121.335 79.395 180)
+    (at 121.995 79.285 180)
     (descr "Through hole angled pin header, 1x03, 1.27mm pitch, 4.0mm pin length, single row")
     (tags "Through hole angled pin header THT 1x03 1.27mm single row")
@@
   (gr_arc (start 120 93.55) (mid 115.947004 91.684798) (end 114.4 87.5)
     (stroke (width 0.05) (type default)) (layer "Edge.Cuts"))
-  (gr_text "T" (at 144.57 84.99) (layer "F.Cu")
-    (effects (font (size 1.5 1.5) (thickness 0.3) bold) (justify left bottom))
-  )
-  (gr_text "Maëna CHARBONNIER" (at 119.05 93.47) (layer "F.Cu")
-    (effects (font (size 1.5 1.5) (thickness 0.3) bold) (justify left bottom))
-  )
-  (gr_text "B" (at 145.18 89.02) (layer "B.Cu")
-    (effects (font (size 1.5 1.5) (thickness 0.3) bold) (justify left bottom))
-  )
+  (segment (start 128.3 78.365) (end 127.225 78.365) (width 0.3) (layer "F.Cu") (net 1))
+  (segment (start 127.225 78.365) (end 127.075 78.215) (width 0.3) (layer "F.Cu") (net 1))
   (segment (start 127.075 78.215) (end 127.075 73.205) (width 0.3) (layer "F.Cu") (net 1))
   (segment (start 128.43 71.85) (end 125.2 68.62) (width 0.3) (layer "F.Cu") (net 1))
   (segment (start 125.2 68.62) (end 125.2 64) (width 0.3) (layer "F.Cu") (net 1))
   (segment (start 127.075 73.205) (end 128.43 71.85) (width 0.3) (layer "F.Cu") (net 1))
-  (segment (start 128.3 78.365) (end 127.225 78.365) (width 0.3) (layer "F.Cu") (net 1))
-  (segment (start 127.225 78.365) (end 127.075 78.215) (width 0.3) (layer "F.Cu") (net 1))
   (segment (start 139.2 77) (end 139.105 77.095) (width 0.5) (layer "F.Cu") (net 2))
   (segment (start 128.8 64) (end 130.15 62.65) (width 0.5) (layer "F.Cu") (net 2))
@@
   (segment (start 131.19 89.95) (end 131.19 79.73) (width 0.5) (layer "B.Cu") (net 2))
   (segment (start 134.73 71.85) (end 134.73 73.91) (width 0.3) (layer "F.Cu") (net 3))
-  (segment (start 134.73 73.91) (end 129.005 79.635) (width 0.3) (layer "F.Cu") (net 3))
+  (segment (start 129.04 79.6) (end 127.45 79.6) (width 0.3) (layer "F.Cu") (net 3))
   (segment (start 136.28 67.46) (end 136.28 70.3) (width 0.3) (layer "F.Cu") (net 3))
+  (segment (start 134.73 73.91) (end 129.04 79.6) (width 0.3) (layer "F.Cu") (net 3))
   (segment (start 132.82 64) (end 136.28 67.46) (width 0.3) (layer "F.Cu") (net 3))
   (segment (start 136.28 70.3) (end 134.73 71.85) (width 0.3) (layer "F.Cu") (net 3))
   (segment (start 122.702106 76.745) (end 128.94 82.982894) (width 0.5) (layer "F.Cu") (net 4))
-  (segment (start 128.3 77.095) (end 128.3 76.295) (width 0.5) (layer "F.Cu") (net 4))
   (segment (start 128.94 87.42) (end 128.3 86.78) (width 0.5) (layer "F.Cu") (net 4))
   (segment (start 128.3 74.56) (end 128.6 74.26) (width 0.5) (layer "F.Cu") (net 4))
@@
   (segment (start 144.85 64.652384) (end 144.85 74.95) (width 0.5) (layer "F.Cu") (net 4))
   (segment (start 123.235 76.745) (end 123.35 76.63) (width 0.5) (layer "F.Cu") (net 4))
-  (segment (start 128.3 76.0755) (end 128.0945 75.87) (width 0.5) (layer "F.Cu") (net 4))
   (segment (start 142.047616 61.85) (end 144.85 64.652384) (width 0.5) (layer "F.Cu") (net 4))
   (segment (start 128.3 77.095) (end 128.3 74.56) (width 0.5) (layer "F.Cu") (net 4))
@@
   (segment (start 124.618629 61.85) (end 142.047616 61.85) (width 0.5) (layer "F.Cu") (net 4))
   (segment (start 123.35 63.118629) (end 124.618629 61.85) (width 0.5) (layer "F.Cu") (net 4))
-  (segment (start 128.3 77.095) (end 128.3 76.0755) (width 0.5) (layer "F.Cu") (net 4))
   (segment (start 128.3 86.78) (end 128.3 80.905) (width 0.5) (layer "F.Cu") (net 4))
-  (segment (start 128.3 76.295) (end 128.295 76.29) (width 0.5) (layer "F.Cu") (net 4))
   (via (at 123.35 73.05) (size 1.2) (drill 0.6) (layers "F.Cu" "B.Cu") (net 4))
   (via (at 129.47 73.97) (size 1.2) (drill 0.6) (layers "F.Cu" "B.Cu") (net 4))
-  (via (at 128.0945 75.87) (size 1.2) (drill 0.6) (layers "F.Cu" "B.Cu") (net 4))
-  (segment (start 127.1095 76.855) (end 121.335 76.855) (width 0.5) (layer "B.Cu") (net 4))
   (segment (start 124.27 73.97) (end 123.35 73.05) (width 0.5) (layer "B.Cu") (net 4))
   (segment (start 129.47 73.97) (end 124.27 73.97) (width 0.5) (layer "B.Cu") (net 4))
-  (segment (start 128.0945 75.87) (end 127.1095 76.855) (width 0.5) (layer "B.Cu") (net 4))
+  (segment (start 127.505 76.785) (end 127.57 76.85) (width 0.5) (layer "B.Cu") (net 4))
   (zone (net 2) (net_name "GND") (layer "F.Cu") (hatch edge 0.5)
     (connect_pads (clearance 0.5))
