File: Hardware/PCB_IR/cohoma-backups/cohoma-2023-05-15_150048/cohoma-backups/cohoma-2023-05-03_234336/cohoma.kicad_sch (KiCad schematic)
At the start: 11 parts, among them J2 Conn_01x03, U1 MCP2120-I/P, U2 TSOP75338WTT, Y1 ABLS-7.3728MHz-20-B-3-H-T

Commit message: pcb
Parts:
- C1, C2, C3: footprint Capacitor_SMD:C_0201_0603Metric_Pad0.64x0.40mm_HandSolder -> Capacitor_SMD:CP_Elec_4x5.4
- U1: footprint Package_SO:SOIC-14_3.9x8.7mm_P1.27mm -> Package_SO:SOIC-8-N7_3.9x4.9mm_P1.27mm
- U2: footprint Package_SO:TSOP753TT -> Capacitor_SMD:CP_Elec_4x5.4
Changed lines of the file:
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@@
       (effects (font (size 1.27 1.27)) (justify left))
     )
-    (property "Footprint" "Capacitor_SMD:C_0201_0603Metric_Pad0.64x0.40mm_HandSolder" (at 229.5652 59.69 0)
+    (property "Footprint" "Capacitor_SMD:CP_Elec_4x5.4" (at 229.5652 59.69 0)
       (effects (font (size 1.27 1.27)) hide)
     )
@@
       (effects (font (size 1.27 1.27)) (justify left))
     )
-    (property "Footprint" "Capacitor_SMD:C_0201_0603Metric_Pad0.64x0.40mm_HandSolder" (at 210.5152 142.24 0)
+    (property "Footprint" "Capacitor_SMD:CP_Elec_4x5.4" (at 210.5152 142.24 0)
       (effects (font (size 1.27 1.27)) hide)
     )
@@
       (effects (font (size 1.27 1.27)) (justify left))
     )
-    (property "Footprint" "Capacitor_SMD:C_0201_0603Metric_Pad0.64x0.40mm_HandSolder" (at 258.7752 60.96 0)
+    (property "Footprint" "Capacitor_SMD:CP_Elec_4x5.4" (at 258.7752 60.96 0)
       (effects (font (size 1.27 1.27)) hide)
     )
@@
       (effects (font (size 1.27 1.27)))
     )
-    (property "Footprint" "Package_SO:SOIC-14_3.9x8.7mm_P1.27mm" (at 55.88 60.96 0)
+    (property "Footprint" "Package_SO:SOIC-8-N7_3.9x4.9mm_P1.27mm" (at 55.88 60.96 0)
       (effects (font (size 1.27 1.27)) (justify bottom) hide)
     )
@@
       (effects (font (size 1.524 1.524)))
     )
-    (property "Footprint" "Package_SO:TSOP753TT" (at 175.26 149.606 0)
+    (property "Footprint" "Capacitor_SMD:CP_Elec_4x5.4" (at 175.26 149.606 0)
       (effects (font (size 1.524 1.524)) hide)
     )
