File: Hardware/PCB_BuckBoost/pcb_v3/pcb_v3.kicad_sch (KiCad schematic)
At the start: 44 parts, among them J1 Conn_01x02, J2 Conn_01x02, J3 Conn_01x02, J4 Conn_01x02, U1 MIC3172YM, U2 MIC3172YM

Commit message: PCB_VB (il reste une erreur au niveau du F.cu)
Parts:
- R8: value 1k -> 183
- R8: value 5,5k -> 1k
- R8: value 1,5k -> 277
- R8: value 3.6k -> 666
Connections:
- net +3.3V: now also R8.1
- net +5V: now also R8.1
- net Routeur: now also R8.1
- net +15V renamed +12V
- net +12V: no longer R8.1, R8.1, R8.1
