File: Hardware/PCB_BuckBoost/pcb_v3/pcb_v3.kicad_pcb (KiCad board)
At the start: 2 copper layers, 43 x 69 mm, 42 parts, among them J1 Conn_01x02, J2 Conn_01x02, J3 Conn_01x02, J4 Conn_01x02, U1 MIC3172YM, U2 MIC3172YM

Commit message: PCB V3 presque fini (il manque quelques tracks)
Parts:
- added C1: 0.47u, Capacitor_SMD:C_0603_1608Metric, F.Cu at (145.7, 85.6)
- added C10: 22uF, Capacitor_SMD:CP_Elec_5x5.4, F.Cu at (127.0, 106.9)
- added C2: 100uF, Capacitor_SMD:CP_Elec_6.3x7.7, F.Cu at (122.8, 66.3)
- added C3: 2.2 µF, Capacitor_SMD:C_0603_1608Metric_Pad1.08x0.95mm_HandSolder, F.Cu at (139.0, 66.8)
- added C4: 1 µF, Capacitor_SMD:C_0603_1608Metric_Pad1.08x0.95mm_HandSolder, F.Cu at (138.9, 73.3)
- added C5: 0.47u, Capacitor_SMD:C_0603_1608Metric_Pad1.08x0.95mm_HandSolder, F.Cu at (145.7, 79.4)
- added C6: 1 µF, Capacitor_SMD:C_0603_1608Metric_Pad1.08x0.95mm_HandSolder, F.Cu at (142.8, 72.3)
- added C7: 330uF, Capacitor_SMD:CP_Elec_10x10.5, F.Cu at (123.8, 81.8)
- added C8: 1µF, Capacitor_SMD:C_0603_1608Metric_Pad1.08x0.95mm_HandSolder, F.Cu at (143.4, 97.5)
- added C9: 470uF, Capacitor_SMD:CP_Elec_10x10.5, F.Cu at (140.8, 106.9)
- added D1: 1N4148, Diode_SMD:D_SOD-123F, F.Cu at (130.6, 66.3)
- added D2: FSV330AF, Footprints_Balise:Diode_Shottky, F.Cu at (124.0, 67.2)
- added D3: 1N4148, Diode_SMD:D_SOD-323F, F.Cu at (142.9, 70.2)
- added D4: FSV330AF, Footprints_Balise:Diode_Shottky, F.Cu at (127.3, 102.0)
- added D5: LED, LED_SMD:LED_0603_1608Metric_Pad1.05x0.95mm_HandSolder, F.Cu at (154.8, 92.5)
- added D6: LED, LED_SMD:LED_0603_1608Metric_Pad1.05x0.95mm_HandSolder, F.Cu at (154.8, 95.1)
- added D7: LED, LED_SMD:LED_0603_1608Metric_Pad1.05x0.95mm_HandSolder, F.Cu at (154.8, 97.7)
- added D8: LED, LED_SMD:LED_0603_1608Metric_Pad1.05x0.95mm_HandSolder, F.Cu at (154.8, 100.3)
- added H1: MountingHole_Pad, MountingHole:MountingHole_3.2mm_M3_Pad_Via, F.Cu at (120.2, 115.0)
- added H2: MountingHole_Pad, MountingHole:MountingHole_3.2mm_M3_Pad_Via, F.Cu at (120.1, 56.6)
- added H3: MountingHole_Pad, MountingHole:MountingHole_3.2mm_M3_Pad_Via, F.Cu at (152.5, 56.8)
- added H4: MountingHole_Pad, MountingHole:MountingHole_3.2mm_M3_Pad_Via, F.Cu at (152.8, 115.8)
- added J1: Conn_01x02, Connector_JST:JST_XH_B2B-XH-A_1x02_P2.50mm_Vertical, F.Cu at (152.5, 67.1)
- added J2: Conn_01x02, Connector_JST:JST_XH_B2B-XH-A_1x02_P2.50mm_Vertical, F.Cu at (152.4, 77.5)
- added J3: Conn_01x02, Connector_JST:JST_XH_B2B-XH-A_1x02_P2.50mm_Vertical, F.Cu at (152.3, 87.7)
- added J4: Conn_01x02, Connector_JST:JST_XH_B2B-XH-A_1x02_P2.50mm_Vertical, F.Cu at (152.3, 108.2)
- added L1: 100 µH, Inductor_SMD:L_Wuerth_WE-PD-Typ-LS, F.Cu at (136.6, 81.9)
- added L2: 100 µH, Inductor_SMD:L_Wuerth_WE-PD-Typ-LS, F.Cu at (123.8, 97.1)
- added PS1: BU33SD5WG-TR, Footprints_Balise:PS1, F.Cu at (146.7, 77.6)
- added R1: 470, Resistor_SMD:R_0603_1608Metric_Pad0.98x0.95mm_HandSolder, F.Cu at (138.9, 71.7)
- added R10: 100, Resistor_SMD:R_0603_1608Metric_Pad0.98x0.95mm_HandSolder, F.Cu at (117.7, 89.1)
- added R11: 3.6k, Resistor_SMD:R_0603_1608Metric_Pad0.98x0.95mm_HandSolder, F.Cu at (150.5, 95.2)
- added R12: 1,5k, Resistor_SMD:R_0603_1608Metric_Pad0.98x0.95mm_HandSolder, F.Cu at (150.5, 97.7)
- added R13: 1k, Resistor_SMD:R_0603_1608Metric_Pad0.98x0.95mm_HandSolder, F.Cu at (150.5, 100.2)
- added R2: 1.2 k, Resistor_SMD:R_0603_1608Metric_Pad0.98x0.95mm_HandSolder, F.Cu at (138.9, 68.6)
- added R3: 3.7k, Resistor_SMD:R_0603_1608Metric_Pad0.98x0.95mm_HandSolder, F.Cu at (138.9, 70.2)
- added R4: 10Ω, Resistor_SMD:R_0603_1608Metric_Pad0.98x0.95mm_HandSolder, F.Cu at (142.8, 68.3)
- added R5: 1k, Resistor_SMD:R_0603_1608Metric_Pad0.98x0.95mm_HandSolder, F.Cu at (143.4, 95.5)
- added R6: 10.7k, Resistor_SMD:R_0603_1608Metric_Pad0.98x0.95mm_HandSolder, F.Cu at (143.4, 91.3)
- added R7: 1.24k, Resistor_SMD:R_0603_1608Metric_Pad0.98x0.95mm_HandSolder, F.Cu at (143.4, 93.4)
- added R8: 5,5k, Resistor_SMD:R_0603_1608Metric_Pad0.98x0.95mm_HandSolder, F.Cu at (150.6, 92.4)
- added R9: 100, Resistor_SMD:R_0603_1608Metric_Pad0.98x0.95mm_HandSolder, F.Cu at (118.3, 73.2)
- added U1: MIC3172YM, Package_SO:SOIC-8-1EP_3.9x4.9mm_P1.27mm_EP2.29x3mm, F.Cu at (132.2, 70.8)
- added U2: MIC3172YM, Package_SO:SOIC-8-1EP_3.9x4.9mm_P1.27mm_EP2.29x3mm, F.Cu at (136.9, 94.1)
- R6: value 10.7 -> 10.7k
Connections:
- C5 pad 1: (no net) -> +5V
- J1 pad 2: (no net) -> +5V
- PS1 pad 5: (no net) -> +5V
- R11 pad 1: (no net) -> +5V
Routing:
- net +5V: track 80.9 -> 165.9 mm, vias 4 -> 6
- net Routeur: track 0.00 -> 70.4 mm, vias 0 -> 2
- net (no net): track 194.6 -> 156.1 mm, vias 22 -> 20
- net +3.3V: track 0.00 -> 19.8 mm
- net +15V: track 0.00 -> 17.9 mm
- net Net-(D1-K): track 11.0 -> 22.6 mm
- net Net-(D4-A): track 0.00 -> 10.0 mm
- net Net-(U2-FB): track 0.00 -> 7.24 mm
- net Net-(U1-FB): track 0.00 -> 7.20 mm
- net Net-(D2-K): track 44.6 -> 50.6 mm
- net Net-(U2-COMP): track 0.00 -> 3.43 mm
- net Net-(D6-A): track 0.00 -> 2.49 mm
- net Net-(D8-A): track 0.00 -> 2.49 mm
- net Net-(D7-A): track 0.00 -> 2.46 mm
- net Net-(D5-A): track 0.00 -> 2.44 mm
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Other:
- board size 43 x 69 mm -> 101.8 x 69.3 mm

Commit message: PCB_VB (il reste une erreur au niveau du F.cu)
Parts:
- removed the C1 at (204.0, 84.3)
- removed the C10 at (185.7, 106.5)
- removed the C2 at (180.3, 66.2)
- removed the C3 at (195.1, 66.3)
- removed the C4 at (195.1, 72.3)
- removed the C5 at (204.2, 79.3)
- removed the C6 at (198.8, 71.0)
- removed the C7 at (181.9, 81.3)
- removed the C8 at (200.5, 96.7)
- removed the C9 at (198.7, 104.1)
- removed the D1 at (187.6, 64.8)
- removed the D2 at (181.3, 72.2)
- removed the D3 at (198.8, 69.3)
- removed the D4 at (190.9, 100.7)
- removed the D5 at (214.4, 99.7)
- removed the D6 at (214.4, 95.7)
- removed the D7 at (214.4, 97.7)
- removed the D8 at (214.4, 93.7)
- removed the H1 at (178.5, 115.8)
- removed the H2 at (178.5, 56.8)
- removed the H3 at (211.5, 56.8)
- removed the H4 at (211.5, 115.8)
- removed the J1 at (211.5, 67.2)
- removed the J2 at (211.5, 77.2)
- removed the J3 at (211.5, 87.2)
- removed the J4 at (211.5, 108.8)
- removed the L1 at (194.3, 81.3)
- removed the L2 at (182.5, 96.7)
- removed the PS1 at (204.1, 81.8)
- removed the R1 at (195.1, 70.8)
- removed the R10 at (210.4, 97.7)
- removed the R11 at (210.4, 93.7)
- removed the R2 at (195.1, 67.8)
- removed the R3 at (195.1, 69.3)
- removed the R4 at (198.8, 67.5)
- removed the R5 at (200.5, 95.2)
- removed the R6 at (200.5, 92.2)
- removed the R7 at (200.5, 93.7)
- removed the R8 at (210.4, 99.7)
- removed the R9 at (210.4, 95.7)
- removed the U1 at (189.3, 69.3)
- removed the U2 at (194.9, 93.7)
- R11: value 3.6k -> 666
- R12: value 1,5k -> 277
- R13: value 1k -> 183
- R8: value 5,5k -> 1k
- moved D2 10.9 mm to (123.3, 78.1), turned to 180 degrees
- moved D8 7.52 mm to (154.9, 92.8)
- moved R13 7.52 mm to (150.6, 92.7)
- moved D5 5.16 mm to (154.7, 97.7)
- moved R8 5.16 mm to (150.5, 97.5)
- moved D6 4.70 mm to (154.7, 99.8)
- moved R11 4.70 mm to (150.5, 99.9)
- moved D7 2.60 mm to (154.8, 95.1)
- moved R12 2.60 mm to (150.6, 95.1)
- moved R9 1.69 mm to (117.8, 74.8), turned to 180 degrees
Connections:
- C10 pad 1: +15V -> +12V
- C2 pad 1: +15V -> +12V
- D1 pad 2: +15V -> +12V
- J4 pad 2: +15V -> +12V
- L2 pad 1: +15V -> +12V
- R11 pad 1: +15V -> +12V
- R12 pad 1: +15V -> +5V
- R13 pad 1: +15V -> +3.3V
- R8 pad 1: +15V -> Routeur
- U1 pad 7: +15V -> +12V
- U2 pad 5: +15V -> +12V
Routing:
- net (no net): track 156.1 -> 0.00 mm, vias 20 -> 0
- net +12V: track 0.00 -> 150.9 mm, vias 0 -> 8
- net +5V: track 165.9 -> 101.6 mm, vias 6 -> 4
- net +15V: track 17.9 -> 0.00 mm
- net +3.3V: track 19.8 -> 35.3 mm, vias 0 -> 2
- net Net-(D1-K): track 22.6 -> 11.6 mm
- net Routeur: track 70.4 -> 75.8 mm, vias 2 -> 5
- net Net-(D3-K): track 3.49 -> 0.00 mm
- net Net-(U1-COMP): track 0.00 -> 3.37 mm
- net Net-(D2-K): track 50.6 -> 53.2 mm
- net Net-(D3-A): track 3.84 -> 1.96 mm
- added copper zone on B.Cu, net GND
- removed copper zone on B.Cu, net (none)
- removed copper zone on F.Cu, net (none)
Other:
- board size 101.8 x 69.3 mm -> 43 x 69 mm
- board text added: "Boost"
- board text added: "Buck"
- board text added: "Cohoma_Balise_V3"

Commit message: PCB V3 fini
Routing:
- net +5V: track 101.6 -> 103.5 mm, vias 4 -> 5
Changed lines of the file:
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@@
     (effects (font (size 1.5 1.5) (thickness 0.3) bold) (justify left bottom mirror))
   )
+  (segment (start 149.779313 85) (end 149.287212 85) (width 1) (layer "F.Cu") (net 2))
   (segment (start 118.7177 80.9211) (end 123.7996 86.003) (width 1) (layer "F.Cu") (net 2))
   (segment (start 124.6078 86.8112) (end 123.7996 86.003) (width 1) (layer "F.Cu") (net 2))
   (segment (start 146.094969 87.9094) (end 144.3482 87.9094) (width 1) (layer "F.Cu") (net 2))
-  (segment (start 150.383 75.0154) (end 150.383 83.621369) (width 1) (layer "F.Cu") (net 2))
   (segment (start 144.3482 87.9094) (end 137.674 87.9094) (width 1) (layer "F.Cu") (net 2))
   (segment (start 147.5486 92.9975) (end 147.5486 91.9226) (width 0.5) (layer "F.Cu") (net 2))
@@
   (segment (start 145.4956 83.4009) (end 144.5384 83.4009) (width 0.5) (layer "F.Cu") (net 2))
   (segment (start 144.5384 85.2046) (end 144.9318 85.598) (width 0.5) (layer "F.Cu") (net 2))
+  (segment (start 150 84.779313) (end 149.779313 85) (width 1) (layer "F.Cu") (net 2))
   (segment (start 137.674 87.9094) (end 136.5758 86.8112) (width 1) (layer "F.Cu") (net 2))
+  (segment (start 150 83) (end 150 84.779313) (width 1) (layer "F.Cu") (net 2))
+  (segment (start 152 81) (end 150 83) (width 1) (layer "F.Cu") (net 2))
   (segment (start 144.5384 81.5213) (end 145.4956 81.5213) (width 0.5) (layer "F.Cu") (net 2))
-  (segment (start 150.383 83.621369) (end 146.094969 87.9094) (width 1) (layer "F.Cu") (net 2))
   (segment (start 144.9318 85.598) (end 144.9318 87.3258) (width 1) (layer "F.Cu") (net 2))
   (segment (start 141.9352 67.31) (end 142.7988 66.4464) (width 0.5) (layer "F.Cu") (net 2))
@@
   (segment (start 141.9352 68.3066) (end 141.9352 67.31) (width 0.5) (layer "F.Cu") (net 2))
   (segment (start 144.5384 83.4009) (end 144.5384 85.2046) (width 0.5) (layer "F.Cu") (net 2))
+  (segment (start 146.377812 87.9094) (end 146.094969 87.9094) (width 1) (layer "F.Cu") (net 2))
   (segment (start 120.7248 89.0778) (end 123.7996 86.003) (width 1) (layer "F.Cu") (net 2))
   (segment (start 145.4956 81.5213) (end 145.5456 81.5713) (width 0.5) (layer "F.Cu") (net 2))
-  (segment (start 152.383 75.0154) (end 150.383 75.0154) (width 1) (layer "F.Cu") (net 2))
+  (segment (start 149.287212 85) (end 146.377812 87.9094) (width 1) (layer "F.Cu") (net 2))
   (segment (start 145.5456 83.3509) (end 145.4956 83.4009) (width 0.5) (layer "F.Cu") (net 2))
   (via (at 146.094969 87.9094) (size 1.2) (drill 0.8) (layers "F.Cu" "B.Cu") (net 2))
+  (via (at 152 81) (size 1.2) (drill 0.8) (layers "F.Cu" "B.Cu") (net 2))
   (via (at 144.3482 87.9094) (size 1.2) (drill 0.8) (layers "F.Cu" "B.Cu") (net 2))
   (via (at 147.5486 91.9226) (size 1.2) (drill 0.8) (layers "F.Cu" "B.Cu") (net 2))
   (via (at 142.7988 66.4464) (size 1.2) (drill 0.8) (layers "F.Cu" "B.Cu") (net 2))
+  (segment (start 154.383 79.617) (end 153 81) (width 1) (layer "B.Cu") (net 2))
   (segment (start 142.7988 66.4464) (end 144.787 68.4346) (width 0.5) (layer "B.Cu") (net 2))
+  (segment (start 153.000767 75.0154) (end 154.383 76.397633) (width 1) (layer "B.Cu") (net 2))
   (segment (start 144.787 87.4706) (end 144.3482 87.9094) (width 0.5) (layer "B.Cu") (net 2))
+  (segment (start 154.383 76.397633) (end 154.383 79.617) (width 1) (layer "B.Cu") (net 2))
+  (segment (start 152.383 75.0154) (end 153.000767 75.0154) (width 1) (layer "B.Cu") (net 2))
   (segment (start 147.5486 89.363031) (end 146.094969 87.9094) (width 0.5) (layer "B.Cu") (net 2))
   (segment (start 147.5486 91.9226) (end 147.5486 89.363031) (width 0.5) (layer "B.Cu") (net 2))
   (segment (start 144.787 68.4346) (end 144.787 87.4706) (width 0.5) (layer "B.Cu") (net 2))
+  (segment (start 153 81) (end 152 81) (width 1) (layer "B.Cu") (net 2))
   (segment (start 134.7216 68.9342) (end 135.5866 68.9342) (width 0.5) (layer "F.Cu") (net 3))
   (segment (start 133.323 67.5356) (end 134.7216 68.9342) (width 0.5) (layer "F.Cu") (net 3))

Commit message: PCB V3 VRAIMENT FINI
Routing:
- net +12V: track 150.9 -> 176.0 mm, vias 8 -> 16
- added copper zone on B.Cu, net +12V
- removed copper zone on B.Cu, net GND
